File: Circuit/Schematics/bottom.brd (EAGLE design)
At the start: 38.1 x 38.1 mm, 53 parts, among them IC1 LM2936MP-3.3, Y1 16 Mhz, Y2 16 Mhz

Commit message: Final P1 boards, ordered on Seeed
Parts:
- removed L3GD20H: L3GD20H, st:LGA16L
- added U$2: L3GD20H, st:LGA16L
- moved C5 1.67 mm to (7.49, 35.1), turned to 270 degrees
- moved C3 0.65 mm to (12.8, 32.4)
- renumbered WIFI_STORAGE to U$3
Connections:
- removed net N$49: L3GD20H.P$7
- removed net N$50: L3GD20H.P$6
- removed net N$54: C3.1, L3GD20H.P$14
- removed net N$58: L3GD20H.P$15
- new net N$11: U$2.P$7
- new net N$12: U$2.P$6
- new net N$22: C3.1, U$2.P$14
- new net N$31: C3.2
- net GND: now also U$2.P$10, U$2.P$11, U$2.P$12, U$2.P$13, U$2.P$8, U$2.P$9; no longer C3.2, L3GD20H.P$10, L3GD20H.P$11, L3GD20H.P$12, L3GD20H.P$13, L3GD20H.P$8, L3GD20H.P$9, R1.2
- net SCL: now also U$2.P$2; no longer L3GD20H.P$2
- net SDA: now also U$2.P$3; no longer L3GD20H.P$3
- net SDO: now also U$2.P$4; no longer L3GD20H.P$4
- net VDD: now also U$2.P$1, U$2.P$15, U$2.P$16, U$2.P$5; no longer L3GD20H.P$1, L3GD20H.P$16, L3GD20H.P$5
Routing:
- net N$22: track 0.00 -> 23.0 mm, vias 0 -> 1
- net N$54: track 22.0 -> 0.00 mm, vias 1 -> 0
- net GND: track 230.3 -> 219.6 mm
- net TX_W: track 47.5 -> 42.6 mm
- net RX_W: track 46.9 -> 42.3 mm
- net SD-D1: track 21.7 -> 17.8 mm
- net VDD: track 205.3 -> 207.5 mm
- net VRAW: vias 3 -> 2
