File: Circuit/Schematics/bottom.sch (EAGLE design)
At the start: 53 parts, among them IC1 LM2936MP-3.3, Y1 16 Mhz, Y2 16 Mhz

Commit message: Final P1 boards, ordered on Seeed
Parts:
- removed L3GD20H: L3GD20H, st:L3GD20H
- removed WIFI_STORAGE: 25Q40, wifi:25Q40
- added U$2: L3GD20H, st:L3GD20H
- added U$3: 25Q40, wifi:25Q40
Connections:
- removed net N$49: L3GD20H.INT1
- removed net N$50: L3GD20H.DRDY/INT2
- removed net N$54: C3.1, L3GD20H.CAP
- new net N$11: U$2.INT1
- new net N$12: U$2.DRDY/INT2
- new net N$22: C3.1, U$2.CAP
- new net N$31: C3.2
- net GND: now also U$2.DEN, U$2.GND, U$2.RES1, U$2.RES2, U$2.RES3, U$3.GND; no longer C3.2, L3GD20H.DEN, L3GD20H.GND, L3GD20H.RES1, L3GD20H.RES2, L3GD20H.RES3, R1.2, WIFI_STORAGE.GND
- net SCL: now also U$2.SCL/SPC; no longer L3GD20H.SCL/SPC
- net SD-CLK: now also U$3.CLK; no longer WIFI_STORAGE.CLK
- net SD-CMD: now also U$3.CS#; no longer WIFI_STORAGE.CS#
- net SD-D0: now also U$3.DO; no longer WIFI_STORAGE.DO
- net SD-D1: now also U$3.DIO; no longer WIFI_STORAGE.DIO
- net SD-D2: now also U$3.HOLD#; no longer WIFI_STORAGE.HOLD#
- net SD-D3: now also U$3.WP#; no longer WIFI_STORAGE.WP#
- net SDA: now also U$2.SDA/SDI; no longer L3GD20H.SDA/SDI
- net SDO: now also U$2.SDO; no longer L3GD20H.SDO
- net VDD: now also U$2.CS, U$2.RES4, U$2.VDD, U$2.VDD_IO, U$3.VCC; no longer L3GD20H.CS, L3GD20H.RES4, L3GD20H.VDD, L3GD20H.VDD_IO, WIFI_STORAGE.VCC
Other:
- moved on the sheet: C5
