File: Circuit/Schematics/top.brd (EAGLE design)
At the start: 38.1 x 38.1 mm, 36 parts, among them Y1 16 MHz, Y2 32.768 kHz

Commit message: Final P1 boards, ordered on Seeed
Parts:
- removed Y2: 32.768 kHz, SparkFun-FreqCtrl:CRYSTAL-SMD-5X3
Connections:
- net N$10 renamed D+
- net N$18 renamed D-
- removed net N$23: U$2.19, Y2.3
- removed net N$24: U$2.20, Y2.1
Routing:
- net N$23: track 12.7 -> 0.00 mm
- net N$24: track 2.93 -> 0.00 mm
Changed lines of the file:
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@@
 <text x="33.528" y="8.382" size="0.8128" layer="25">TX</text>
 <text x="37.338" y="3.81" size="1.778" layer="25" rot="R90">P1</text>
+<polygon width="0.4064" layer="41">
+<vertex x="27.178" y="8.382"/>
+<vertex x="26.416" y="8.382"/>
+<vertex x="26.416" y="4.064"/>
+<vertex x="26.416" y="3.556"/>
+<vertex x="33.782" y="3.556"/>
+<vertex x="33.782" y="8.382"/>
+<vertex x="26.416" y="8.382"/>
+</polygon>
 </plain>
 <attributes>
@@
 <attribute name="PROD_ID" value="XTAL-08218" x="30.48" y="6.096" size="1.778" layer="27" rot="R180" display="off"/>
 </element>
-<element name="Y2" library="SparkFun-FreqCtrl" package="CRYSTAL-SMD-5X3" value="32.768 kHz" x="20.828" y="6.096" rot="R180">
-<attribute name="PROD_ID" value="XTAL-08218" x="20.828" y="6.096" size="1.778" layer="27" rot="R180" display="off"/>
-</element>
 <element name="FUSE" library="SparkFun-PowerIC" package="0603" value="PTC0603" x="29.972" y="36.068" smashed="yes">
 <attribute name="NAME" x="29.083" y="36.83" size="0.4064" layer="25" font="vector"/>
@@
 <contactref element="FERRITE3" pad="1"/>
 <contactref element="JP2" pad="2"/>
-<polygon width="0.254" layer="16">
+<polygon width="0.254" layer="16" isolate="0.381">
 <vertex x="-71.374" y="115.824"/>
 <vertex x="-77.724" y="115.824"/>
@@
 <vertex x="-71.374" y="114.3"/>
 </polygon>
-<polygon width="0.254" layer="1">
+<polygon width="0.254" layer="1" isolate="0.381">
 <vertex x="-60.706" y="109.22"/>
 <vertex x="179.324" y="109.22"/>
@@
 <wire x1="17.272" y1="26.67" x2="18.034" y2="27.432" width="0.254" layer="1"/>
 </signal>
-<signal name="N$10">
+<signal name="D+">
 <contactref element="R2" pad="1"/>
 <contactref element="JP1" pad="D+1"/>
@@
 <wire x1="19.05" y1="31.75" x2="19.05" y2="33.343" width="0.254" layer="1"/>
 </signal>
-<signal name="N$18">
+<signal name="D-">
 <contactref element="R3" pad="1"/>
 <contactref element="JP1" pad="D-1"/>
@@
 <wire x1="19.7" y1="31.95" x2="20.828" y2="30.822" width="0.254" layer="1"/>
 </signal>
-<signal name="N$23">
-<contactref element="U$2" pad="19"/>
-<contactref element="Y2" pad="3"/>
-<wire x1="22.6568" y1="9.779" x2="22.6568" y2="8.6868" width="0.254" layer="1"/>
-<wire x1="22.6568" y1="8.6868" x2="22.352" y2="8.382" width="0.254" layer="1"/>
-<wire x1="22.352" y1="8.382" x2="17.272" y2="8.382" width="0.254" layer="1"/>
-<wire x1="17.272" y1="8.382" x2="16.764" y2="7.62" width="0.254" layer="1"/>
-<wire x1="16.764" y1="7.62" x2="16.764" y2="5.334" width="0.254" layer="1"/>
-<wire x1="16.764" y1="5.334" x2="17.78" y2="4.318" width="0.254" layer="1"/>
-<wire x1="17.78" y1="4.318" x2="18.35" y2="4.318" width="0.254" layer="1"/>
-<wire x1="18.35" y1="4.318" x2="18.978" y2="4.946" width="0.254" layer="1"/>
-</signal>
-<signal name="N$24">
-<contactref element="Y2" pad="1"/>
-<contactref element="U$2" pad="20"/>
-<wire x1="23.1394" y1="9.779" x2="23.1394" y2="8.4074" width="0.254" layer="1"/>
-<wire x1="23.1394" y1="8.4074" x2="22.606" y2="7.874" width="0.254" layer="1"/>
-<wire x1="22.606" y1="7.874" x2="22.606" y2="7.174" width="0.254" layer="1"/>
-<wire x1="22.606" y1="7.174" x2="22.678" y2="7.246" width="0.254" layer="1"/>
-</signal>
 <signal name="N$25">
