File: Circuit/Schematics/top.sch (EAGLE design)
At the start: 36 parts, among them Y1 16 MHz, Y2 32.768 kHz

Commit message: Final P1 boards, ordered on Seeed
Parts:
- removed Y2: 32.768 kHz, SparkFun-FreqCtrl:CRYSTAL5X3
Connections:
- net N$10 renamed D+
- net N$18 renamed D-
- removed net N$23: U$2.XTAL32, Y2.2
- removed net N$24: U$2.EXTAL32, Y2.1
Changed lines of the file:
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@@
 <part name="FERRITE3" library="inductors" deviceset="BLM15H" device="" technology="B121SN1"/>
 <part name="Y1" library="SparkFun-FreqCtrl" deviceset="CRYSTAL" device="5X3" value="16 MHz"/>
-<part name="Y2" library="SparkFun-FreqCtrl" deviceset="CRYSTAL" device="5X3" value="32.768 kHz"/>
 <part name="D6" library="SparkFun-DiscreteSemi" deviceset="DIODE" device="BAS16" value="1A"/>
 <part name="D8" library="SparkFun-DiscreteSemi" deviceset="DIODE" device="BAS16" value="1A"/>
@@
 <instance part="FERRITE3" gate="G$1" x="30.48" y="137.16"/>
 <instance part="Y1" gate="G$1" x="111.76" y="78.74" rot="R90"/>
-<instance part="Y2" gate="G$1" x="101.6" y="106.68" rot="R90"/>
 <instance part="D6" gate="G$1" x="55.88" y="127" rot="R270"/>
 <instance part="D8" gate="G$1" x="91.44" y="175.26" rot="R270"/>
@@
 </segment>
 </net>
-<net name="N$10" class="0">
+<net name="D+" class="0">
 <segment>
 <pinref part="R2" gate="G$1" pin="1"/>
@@
 </segment>
 </net>
-<net name="N$18" class="0">
+<net name="D-" class="0">
 <segment>
 <pinref part="R3" gate="G$1" pin="1"/>
@@
 </segment>
 </net>
-<net name="N$23" class="0">
-<segment>
-<pinref part="U$2" gate="G$1" pin="XTAL32"/>
-<pinref part="Y2" gate="G$1" pin="2"/>
-<wire x1="111.76" y1="109.22" x2="101.6" y2="109.22" width="0.1524" layer="91"/>
-</segment>
-</net>
-<net name="N$24" class="0">
-<segment>
-<pinref part="Y2" gate="G$1" pin="1"/>
-<pinref part="U$2" gate="G$1" pin="EXTAL32"/>
-<wire x1="101.6" y1="104.14" x2="111.76" y2="104.14" width="0.1524" layer="91"/>
-</segment>
-</net>
