File: Circuit/P1R2/key.sch (EAGLE design)
At the start: 8 parts, among them J1 1981584-1, U3 MINI54TAN

Commit message: Forum boards done
Parts:
- removed JP1: (no value), SparkFun-Connectors:M07
- added JP2: M100.1, umich:M100.1
- renumbered C15 to C5
Connections:
- net 3.3V: now also JP2.10
- net GND: now also JP2.1
- net ID: now also JP2.5; no longer JP1.3
- net P0.1: now also JP2.8; no longer JP1.6
- net RESET_B: now also JP2.9; no longer JP1.7
- net SWD_CLK: now also JP2.7; no longer JP1.5
- net SWD_DIO: now also JP2.6; no longer JP1.4
- net USB_D_N: now also JP2.3; no longer JP1.1
- net USB_D_P: now also JP2.4; no longer JP1.2
- net VCC: now also JP2.2
Changed lines of the file:
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@@
 <part name="U$14" library="microbuilder" deviceset="GND" device=""/>
 <part name="U$18" library="microbuilder" deviceset="GND" device=""/>
-<part name="C15" library="appfruits" deviceset="CAPACITOR" device="-0.1UF" value="0.1uF"/>
+<part name="C5" library="appfruits" deviceset="CAPACITOR" device="-0.1UF" value="0.1uF"/>
 <part name="PROGRAM" library="SparkFun-Electromechanical" deviceset="SWITCH-MOMENTARY-2" device="-SMD-1101NE" value="Program">
 <attribute name="MF" value="C&amp;K Components"/>
@@
 </part>
 <part name="SUPPLY1" library="SparkFun-Aesthetics" deviceset="VCC" device=""/>
-<part name="JP1" library="SparkFun-Connectors" deviceset="M07" device=""/>
+<part name="JP2" library="umich" deviceset="M10" device="0.1"/>
 </parts>
 <sheets>
@@
 <instance part="U$14" gate="G$1" x="30.48" y="-45.72"/>
 <instance part="U$18" gate="G$1" x="76.2" y="-45.72"/>
-<instance part="C15" gate="G$1" x="76.2" y="-33.02"/>
+<instance part="C5" gate="G$1" x="76.2" y="-33.02"/>
 <instance part="PROGRAM" gate="G$1" x="20.32" y="-17.78" rot="R90">
 <attribute name="MF" x="20.32" y="-17.78" size="1.778" layer="96" rot="R90" display="off"/>
@@
 <instance part="RN1" gate="B" x="43.18" y="66.04"/>
 <instance part="SUPPLY1" gate="G$1" x="68.58" y="76.2"/>
-<instance part="JP1" gate="G$1" x="132.08" y="33.02" rot="R180"/>
+<instance part="JP2" gate="G$1" x="157.48" y="35.56" rot="R180"/>
 </instances>
 <busses>
@@
 </segment>
 <segment>
-<pinref part="C15" gate="G$1" pin="2"/>
+<pinref part="C5" gate="G$1" pin="2"/>
 <pinref part="U$18" gate="G$1" pin="GND"/>
 <wire x1="76.2" y1="-35.56" x2="76.2" y2="-43.18" width="0.1524" layer="91"/>
@@
 <wire x1="33.02" y1="53.34" x2="40.64" y2="53.34" width="0.1524" layer="91"/>
 <wire x1="40.64" y1="53.34" x2="40.64" y2="50.8" width="0.1524" layer="91"/>
+</segment>
+<segment>
+<pinref part="JP2" gate="G$1" pin="1"/>
+<wire x1="149.86" y1="48.26" x2="147.32" y2="48.26" width="0.1524" layer="91"/>
 </segment>
 </net>
@@
 <wire x1="-10.16" y1="22.86" x2="-10.16" y2="43.18" width="0.1524" layer="91"/>
 </segment>
+<segment>
+<pinref part="JP2" gate="G$1" pin="10"/>
+<wire x1="149.86" y1="25.4" x2="147.32" y2="25.4" width="0.1524" layer="91"/>
+</segment>
 </net>
 <net name="SWD_DIO" class="0">
@@
 </segment>
 <segment>
-<pinref part="JP1" gate="G$1" pin="4"/>
-<wire x1="127" y1="30.48" x2="121.92" y2="30.48" width="0.1524" layer="91"/>
+<pinref part="JP2" gate="G$1" pin="6"/>
+<wire x1="149.86" y1="35.56" x2="147.32" y2="35.56" width="0.1524" layer="91"/>
 </segment>
 </net>
@@
 </segment>
 <segment>
-<pinref part="JP1" gate="G$1" pin="5"/>
-<wire x1="127" y1="27.94" x2="121.92" y2="27.94" width="0.1524" layer="91"/>
+<pinref part="JP2" gate="G$1" pin="7"/>
+<wire x1="149.86" y1="33.02" x2="147.32" y2="33.02" width="0.1524" layer="91"/>
 </segment>
 </net>
@@
 </segment>
 <segment>
-<pinref part="JP1" gate="G$1" pin="6"/>
-<wire x1="127" y1="25.4" x2="121.92" y2="25.4" width="0.1524" layer="91"/>
+<pinref part="JP2" gate="G$1" pin="8"/>
+<wire x1="149.86" y1="30.48" x2="147.32" y2="30.48" width="0.1524" layer="91"/>
 </segment>
 </net>
@@
 </segment>
 <segment>
-<pinref part="JP1" gate="G$1" pin="7"/>
-<wire x1="127" y1="22.86" x2="121.92" y2="22.86" width="0.1524" layer="91"/>
+<pinref part="JP2" gate="G$1" pin="9"/>
+<wire x1="149.86" y1="27.94" x2="147.32" y2="27.94" width="0.1524" layer="91"/>
 </segment>
 </net>
@@
 <segment>
 <pinref part="U3" gate="G$1" pin="LDOCAP"/>
-<pinref part="C15" gate="G$1" pin="1"/>
+<pinref part="C5" gate="G$1" pin="1"/>
 <wire x1="68.58" y1="5.08" x2="76.2" y2="5.08" width="0.1524" layer="91"/>
 <wire x1="76.2" y1="5.08" x2="76.2" y2="-27.94" width="0.1524" layer="91"/>
@@
 </segment>
 <segment>
-<pinref part="JP1" gate="G$1" pin="2"/>
-<wire x1="127" y1="35.56" x2="121.92" y2="35.56" width="0.1524" layer="91"/>
+<pinref part="JP2" gate="G$1" pin="4"/>
+<wire x1="149.86" y1="40.64" x2="147.32" y2="40.64" width="0.1524" layer="91"/>
 </segment>
 </net>
@@
 </segment>
 <segment>
-<pinref part="JP1" gate="G$1" pin="1"/>
-<wire x1="127" y1="38.1" x2="121.92" y2="38.1" width="0.1524" layer="91"/>
+<pinref part="JP2" gate="G$1" pin="3"/>
+<wire x1="149.86" y1="43.18" x2="147.32" y2="43.18" width="0.1524" layer="91"/>
 </segment>
 </net>
@@
 </segment>
 <segment>
-<pinref part="JP1" gate="G$1" pin="3"/>
-<wire x1="127" y1="33.02" x2="121.92" y2="33.02" width="0.1524" layer="91"/>
+<pinref part="JP2" gate="G$1" pin="5"/>
+<wire x1="149.86" y1="38.1" x2="147.32" y2="38.1" width="0.1524" layer="91"/>
 </segment>
 </net>
@@
 <pinref part="SUPPLY1" gate="G$1" pin="VCC"/>
 </segment>
-</net>
+<segment>
+<pinref part="JP2" gate="G$1" pin="2"/>
+<wire x1="149.86" y1="45.72" x2="147.32" y2="45.72" width="0.1524" layer="91"/>
+</segment>
+</net>
