File: Circuit/P1R2/patch.sch (EAGLE design)
At the start: 71 parts, among them U1 MK20DX256VLH7, U2 TPS61200, U3 MPU-9250, Y1 32.768KHz, Y2 16Mhz/8pF, Y3 26 Mhz, Y4 16 Mhz

Commit message: Last couple power connections left. Everything else is placed
Parts:
- removed JP6: M100.1, umich:M100.1
- added C26, C28: 0.1uF, appfruits:CAPACITOR-0.1UF
- added C29, C30, C31, C32: 22 pF, appfruits:CAPACITOR-10UF
- added J1: 1981584-1, con-usb:1981584-1
- added L7: 600 Ohm/100 Mhz, appfruits:INDUCTOR-BK2125HM601-T
- added PROGRAM: Program, SparkFun-Electromechanical:SWITCH-MOMENTARY-2-SMD-1101NE
- added RN1: 33, resistor-dil:2R-NEXB34V
- added U4: MINI54TAN, TeensyCustom:MINI54TAN
Connections:
- new net N$10: PROGRAM.2, U4.P5.2
- new net N$11: C26.1, U4.LDOCAP
- new net USB_CON_N: J1.D-, RN1A.1
- new net USB_CON_P: J1.D+, RN1B.1
- new net USB_SHIELD: J1.S1, J1.S2, J1.S3, J1.S4, L7.2
- net 3.3V: now also C28.1, U4.AVDD, U4.VDD; no longer JP6.1
- net GND: now also C26.2, C28.2, C29.1, C30.1, C31.1, C32.1, J1.GND, L7.1, LED2.C, LED3.C, LED4.C, PROGRAM.1, U4.AVSS, U4.P1.4, U4.P2.5, U4.VSS; no longer JP6.10, R15.2, R17.2, R8.2
- net ID: now also J1.ID, U4.P0.0; no longer JP6.6
- net N$27: now also C29.2
- net N$28: now also C30.2
- net N$29: now also C31.2
- net N$30: now also C32.2
- net N$7: now also LED2.A, R8.2; no longer LED2.C, R8.1
- net N$8: now also LED3.A, R15.2; no longer LED3.C, R15.1
- net N$9: now also LED4.A, R17.2; no longer LED4.C, R17.1
- net PTA2: now also U4.P0.1; no longer JP6.3
- net PTB2: now also R8.1; no longer LED2.A
- net PTC2: now also R15.1; no longer LED3.A
- net PTC3: now also R17.1; no longer LED4.A
- net RESET_B: now also U4.P3.2; no longer JP6.2
- net SWD_CLK: now also U4.P0.7; no longer JP6.4
- net SWD_DIO: now also U4.P0.5, U4.P0.6; no longer JP6.5
- net USB_D_N: now also RN1A.2; no longer JP6.8
- net USB_D_P: now also RN1B.2; no longer JP6.7
- net VCC: now also J1.VBUS; no longer JP6.9
Other:
- note added: "Place RN1 as close as possible to USB-Connector!"
- note added: "USB_D+ and USB_D- must be routed as a differential pair. By naming them with _N and _P Eagle automatically routes both traces when placing traces in board layout. It uses the DRU and/or net class values. See EAGLE-Menu Edit->Net classes for the values in this example board"

Commit message: Reversioning, now R1, R2, R3 present
Parts:
- removed C26, C28: 0.1uF, appfruits:CAPACITOR-0.1UF
- removed C29, C30, C31, C32: 22 pF, appfruits:CAPACITOR-10UF
- removed J1: 1981584-1, con-usb:1981584-1
- removed L7: 600 Ohm/100 Mhz, appfruits:INDUCTOR-BK2125HM601-T
- removed LED2, LED3, LED4: (no value), appfruits:LED-GREEN
- removed PROGRAM: Program, SparkFun-Electromechanical:SWITCH-MOMENTARY-2-SMD-1101NE
- removed R15, R17, R8: 330, appfruits:RESISTOR-470
- removed RN1: 33, resistor-dil:2R-NEXB34V
- removed U4: MINI54TAN, TeensyCustom:MINI54TAN
- added JP6: M100.1, umich:M100.1
Connections:
- removed net N$10: PROGRAM.2, U4.P5.2
- removed net N$11: C26.1, U4.LDOCAP
- removed net N$7: LED2.A, R8.2
- removed net N$8: LED3.A, R15.2
- removed net N$9: LED4.A, R17.2
- removed net USB_CON_N: J1.D-, RN1A.1
- removed net USB_CON_P: J1.D+, RN1B.1
- removed net USB_SHIELD: J1.S1, J1.S2, J1.S3, J1.S4, L7.2
- net 3.3V: now also JP6.1; no longer C28.1, U4.AVDD, U4.VDD
- net GND: now also JP6.10; no longer C26.2, C28.2, C29.1, C30.1, C31.1, C32.1, J1.GND, L7.1, LED2.C, LED3.C, LED4.C, PROGRAM.1, U4.AVSS, U4.P1.4, U4.P2.5, U4.VSS
- net ID: now also JP6.6; no longer J1.ID, U4.P0.0
- net N$27: no longer C29.2
- net N$28: no longer C30.2
- net N$29: no longer C31.2
- net N$30: no longer C32.2
- net PTA2: now also JP6.3; no longer U4.P0.1
- net PTB2: no longer R8.1
- net PTC2: no longer R15.1
- net PTC3: no longer R17.1
- net RESET_B: now also JP6.2; no longer U4.P3.2
- net SWD_CLK: now also JP6.4; no longer U4.P0.7
- net SWD_DIO: now also JP6.5; no longer U4.P0.5, U4.P0.6
- net USB_D_N: now also JP6.8; no longer RN1A.2
- net USB_D_P: now also JP6.7; no longer RN1B.2
- net VCC: now also JP6.9; no longer J1.VBUS
Other:
- note removed: "GND"
- note removed: "I2C power"
- note removed: "Place RN1 as close as possible to USB-Connector!"
- note removed: "SCL"
- note removed: "SDA"
- note removed: "USB_D+ and USB_D- must be routed as a differential pair. By naming them with _N and _P Eagle automatically routes both traces when placing traces in board layout. It uses the DRU and/or net class values. See EAGLE-Menu Edit->Net classes for the values in this example board"
