File: Circuit/R3_R4/freckle.brd (EAGLE design)
At the start: 50.8 x 50.8 mm, 75 parts, among them U1 MK20DX256VLH7, U2 TPS61200, U3 MPU-9250, Y1 32.768KHz, Y2 16Mhz/8pF, Y3 26 Mhz, Y4 16 Mhz

Commit message: Single line of breakouts,akouts, with 3 V+, 8 GPIO, 4 GND for R3_R4
Parts:
- removed JP2: (no value), SparkFun-Connectors:1X08
- added JP1: (no value), SparkFun-Connectors:1X15
Connections:
- net 3.3V: now also JP1.13, JP1.14, JP1.15
- net GND: now also JP1.1, JP1.2, JP1.3, JP1.4
- net PTC10: now also JP1.12; no longer JP2.8
- net PTC11: now also JP1.11; no longer JP2.7
- net PTD0: now also JP1.10; no longer JP2.6
- net PTD1: now also JP1.9; no longer JP2.5
- net PTD2: now also JP1.8; no longer JP2.4
- net PTD3: now also JP1.7; no longer JP2.3
- net PTD4: now also JP1.6; no longer JP2.2
- net PTD5: now also JP1.5; no longer JP2.1
Routing:
- net 3.3V: track 157.7 -> 189.3 mm, vias 3 -> 4
- net PTC10: track 23.6 -> 25.1 mm
- net PTD5: track 23.7 -> 22.5 mm
- net PTD4: track 22.7 -> 21.7 mm
- net PTD3: track 21.7 -> 20.8 mm
- net PTD2: track 21.4 -> 20.8 mm
- net PTD1: track 21.4 -> 20.8 mm
- net PTD0: track 21.4 -> 20.8 mm
- net PTC11: track 21.8 -> 22.3 mm
Changed lines of the file:
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@@
 <setting verticaltext="up"/>
 </settings>
-<grid distance="1" unitdist="mil" unit="mil" style="lines" multiple="1" display="yes" altdistance="0.025" altunitdist="inch" altunit="inch"/>
+<grid distance="10" unitdist="mil" unit="mil" style="lines" multiple="1" display="yes" altdistance="0.025" altunitdist="inch" altunit="inch"/>
 <layers>
 <layer number="1" name="Top" color="4" fill="1" visible="yes" active="yes"/>
@@
 <attribute name="MF" value="Kemet" x="24.9428" y="27.3558" size="1.778" layer="27" rot="R90" display="off"/>
 </element>
-<element name="JP2" library="SparkFun-Connectors" package="1X08" value="" x="49.403" y="34.29" rot="R270">
-<attribute name="PROD_ID" value="CONN-08438" x="49.403" y="34.29" size="1.778" layer="27" rot="R270" display="off"/>
-</element>
 <element name="L1" library="appfruits" package="LPS3015" value="2.2uH, 2.1A" x="16.2814" y="43.1038" rot="R90">
 <attribute name="MPN" value="LPS3015-222MRB" x="16.2814" y="43.1038" size="1.778" layer="27" rot="R90" display="off"/>
@@
 </element>
 <element name="R18" library="SparkFun-Resistors" package="0603-RES" value="200" x="18.7706" y="19.7358" rot="R270"/>
+<element name="JP1" library="SparkFun-Connectors" package="1X15" value="" x="49.3776" y="43.18" rot="R270"/>
 </elements>
 <signals>
@@
 <wire x1="33.1724" y1="28.2194" x2="36.2712" y2="25.1206" width="0.6096" layer="16"/>
 <wire x1="36.2712" y1="25.1206" x2="40.8686" y2="25.1206" width="0.6096" layer="16"/>
+<contactref element="JP1" pad="1"/>
+<contactref element="JP1" pad="2"/>
+<contactref element="JP1" pad="3"/>
+<contactref element="JP1" pad="4"/>
 </signal>
 <signal name="N$2">
@@
 <signal name="PTD5">
 <contactref element="U1" pad="62"/>
-<contactref element="JP2" pad="1"/>
 <wire x1="35.135" y1="25.1864" x2="35.135" y2="23.285" width="0.254" layer="1"/>
 <wire x1="35.135" y1="23.285" x2="35.814" y2="22.606" width="0.254" layer="1"/>
 <wire x1="35.814" y1="22.606" x2="41.91" y2="22.606" width="0.254" layer="1"/>
-<wire x1="41.91" y1="22.606" x2="46.482" y2="27.178" width="0.254" layer="1"/>
-<wire x1="46.482" y1="27.178" x2="46.482" y2="31.369" width="0.254" layer="1"/>
-<wire x1="46.482" y1="31.369" x2="49.403" y2="34.29" width="0.254" layer="1"/>
+<wire x1="41.91" y1="22.606" x2="46.736" y2="27.432" width="0.254" layer="1"/>
+<contactref element="JP1" pad="5"/>
+<wire x1="46.736" y1="27.432" x2="46.736" y2="30.3784" width="0.254" layer="1"/>
+<wire x1="46.736" y1="30.3784" x2="49.3776" y2="33.02" width="0.254" layer="1"/>
 </signal>
 <signal name="PTB1">
@@
 <signal name="PTD1">
 <contactref element="U1" pad="58"/>
-<contactref element="JP2" pad="5"/>
 <wire x1="33.135" y1="25.1864" x2="33.135" y2="22.237" width="0.254" layer="1"/>
 <wire x1="33.135" y1="22.237" x2="34.798" y2="20.574" width="0.254" layer="1"/>
-<wire x1="34.798" y1="20.574" x2="45.847" y2="20.574" width="0.254" layer="1"/>
-<wire x1="45.847" y1="20.574" x2="49.403" y2="24.13" width="0.254" layer="1"/>
+<wire x1="34.798" y1="20.574" x2="47.0916" y2="20.574" width="0.254" layer="1"/>
+<contactref element="JP1" pad="9"/>
+<wire x1="47.0916" y1="20.574" x2="49.3776" y2="22.86" width="0.254" layer="1"/>
 </signal>
 <signal name="PTC4">
@@
 <signal name="PTD3">
 <contactref element="U1" pad="60"/>
-<contactref element="JP2" pad="3"/>
 <wire x1="34.135" y1="25.1864" x2="34.135" y2="22.761" width="0.254" layer="1"/>
 <wire x1="34.135" y1="22.761" x2="35.306" y2="21.59" width="0.254" layer="1"/>
 <wire x1="35.306" y1="21.59" x2="42.418" y2="21.59" width="0.254" layer="1"/>
-<wire x1="42.418" y1="21.59" x2="47.498" y2="26.67" width="0.254" layer="1"/>
-<wire x1="47.498" y1="26.67" x2="47.498" y2="27.305" width="0.254" layer="1"/>
-<wire x1="47.498" y1="27.305" x2="49.403" y2="29.21" width="0.254" layer="1"/>
+<wire x1="42.418" y1="21.59" x2="48.768" y2="27.94" width="0.254" layer="1"/>
+<contactref element="JP1" pad="7"/>
+<wire x1="48.768" y1="27.94" x2="49.3776" y2="27.94" width="0.254" layer="1"/>
 </signal>
 <signal name="PTD2">
 <contactref element="U1" pad="59"/>
-<contactref element="JP2" pad="4"/>
 <wire x1="33.635" y1="25.1864" x2="33.635" y2="22.499" width="0.254" layer="1"/>
 <wire x1="33.635" y1="22.499" x2="35.052" y2="21.082" width="0.254" layer="1"/>
 <wire x1="35.052" y1="21.082" x2="42.672" y2="21.082" width="0.254" layer="1"/>
-<wire x1="42.672" y1="21.082" x2="48.26" y2="26.67" width="0.254" layer="1"/>
-<wire x1="48.26" y1="26.67" x2="49.403" y2="26.67" width="0.254" layer="1"/>
+<contactref element="JP1" pad="8"/>
+<wire x1="42.672" y1="21.082" x2="46.99" y2="25.4" width="0.254" layer="1"/>
+<wire x1="46.99" y1="25.4" x2="49.3776" y2="25.4" width="0.254" layer="1"/>
 </signal>
 <signal name="PTD4">
 <contactref element="U1" pad="61"/>
-<contactref element="JP2" pad="2"/>
 <wire x1="34.635" y1="25.1864" x2="34.635" y2="23.023" width="0.254" layer="1"/>
 <wire x1="34.635" y1="23.023" x2="35.56" y2="22.098" width="0.254" layer="1"/>
 <wire x1="35.56" y1="22.098" x2="42.164" y2="22.098" width="0.254" layer="1"/>
-<wire x1="42.164" y1="22.098" x2="46.99" y2="26.924" width="0.254" layer="1"/>
-<wire x1="46.99" y1="26.924" x2="46.99" y2="29.337" width="0.254" layer="1"/>
-<wire x1="46.99" y1="29.337" x2="49.403" y2="31.75" width="0.254" layer="1"/>
+<wire x1="42.164" y1="22.098" x2="47.498" y2="27.432" width="0.254" layer="1"/>
+<contactref element="JP1" pad="6"/>
+<wire x1="47.498" y1="27.432" x2="47.498" y2="28.956" width="0.254" layer="1"/>
+<wire x1="47.498" y1="28.956" x2="49.022" y2="30.48" width="0.254" layer="1"/>
+<wire x1="49.022" y1="30.48" x2="49.3776" y2="30.48" width="0.254" layer="1"/>
 </signal>
 <signal name="PTD7">
@@
 <signal name="PTD0">
 <contactref element="U1" pad="57"/>
-<contactref element="JP2" pad="6"/>
 <wire x1="32.635" y1="25.1864" x2="32.635" y2="21.975" width="0.254" layer="1"/>
 <wire x1="32.635" y1="21.975" x2="34.544" y2="20.066" width="0.254" layer="1"/>
-<wire x1="34.544" y1="20.066" x2="47.879" y2="20.066" width="0.254" layer="1"/>
-<wire x1="47.879" y1="20.066" x2="49.403" y2="21.59" width="0.254" layer="1"/>
+<contactref element="JP1" pad="10"/>
+<wire x1="34.544" y1="20.066" x2="49.1236" y2="20.066" width="0.254" layer="1"/>
+<wire x1="49.1236" y1="20.066" x2="49.3776" y2="20.32" width="0.254" layer="1"/>
 </signal>
 <signal name="PTB17">
@@
 </signal>
 <signal name="PTC11">
-<contactref element="JP2" pad="7"/>
 <contactref element="U1" pad="56"/>
 <wire x1="32.135" y1="25.1864" x2="32.135" y2="21.713" width="0.254" layer="1"/>
 <wire x1="32.135" y1="21.713" x2="34.29" y2="19.558" width="0.254" layer="1"/>
-<wire x1="34.29" y1="19.558" x2="48.895" y2="19.558" width="0.254" layer="1"/>
-<wire x1="48.895" y1="19.558" x2="49.403" y2="19.05" width="0.254" layer="1"/>
+<contactref element="JP1" pad="11"/>
+<wire x1="34.29" y1="19.558" x2="47.5996" y2="19.558" width="0.254" layer="1"/>
+<wire x1="47.5996" y1="19.558" x2="49.3776" y2="17.78" width="0.254" layer="1"/>
 </signal>
 <signal name="PTC10">
-<contactref element="JP2" pad="8"/>
 <contactref element="U1" pad="55"/>
 <wire x1="31.635" y1="25.1864" x2="31.635" y2="21.451" width="0.254" layer="1"/>
 <wire x1="31.635" y1="21.451" x2="34.036" y2="19.05" width="0.254" layer="1"/>
-<wire x1="34.036" y1="19.05" x2="46.863" y2="19.05" width="0.254" layer="1"/>
-<wire x1="46.863" y1="19.05" x2="49.403" y2="16.51" width="0.254" layer="1"/>
+<contactref element="JP1" pad="12"/>
+<wire x1="49.3776" y1="15.24" x2="48.768" y2="15.24" width="0.254" layer="1"/>
+<wire x1="48.768" y1="15.24" x2="47.498" y2="16.51" width="0.254" layer="1"/>
+<wire x1="47.498" y1="16.51" x2="47.498" y2="18.288" width="0.254" layer="1"/>
+<wire x1="47.498" y1="18.288" x2="46.736" y2="19.05" width="0.254" layer="1"/>
+<wire x1="46.736" y1="19.05" x2="34.036" y2="19.05" width="0.254" layer="1"/>
 </signal>
 <signal name="PTC9">
@@
 <wire x1="28.3036" y1="11.0664" x2="27.178" y2="12.192" width="0.254" layer="1"/>
 <wire x1="27.178" y1="12.192" x2="27.178" y2="14.4272" width="0.254" layer="1"/>
-<wire x1="27.178" y1="14.4272" x2="27.178" y2="16.4592" width="0.6096" layer="1"/>
-<wire x1="27.178" y1="16.4592" x2="23.622" y2="20.0152" width="0.6096" layer="1"/>
+<wire x1="27.178" y1="14.4272" x2="27.178" y2="16.256" width="0.6096" layer="1"/>
+<wire x1="26.5176" y1="17.1196" x2="23.622" y2="20.0152" width="0.6096" layer="1"/>
 <wire x1="23.622" y1="20.0152" x2="23.622" y2="23.6474" width="0.6096" layer="1"/>
 <wire x1="23.622" y1="23.6474" x2="23.749" y2="23.7744" width="0.6096" layer="1"/>
@@
 <wire x1="23.749" y1="23.7744" x2="23.749" y2="25.312" width="0.6096" layer="1"/>
 <wire x1="23.749" y1="25.312" x2="24.9428" y2="26.5058" width="0.6096" layer="1"/>
+<contactref element="JP1" pad="13"/>
+<contactref element="JP1" pad="14"/>
+<contactref element="JP1" pad="15"/>
+<wire x1="49.3776" y1="10.16" x2="30.226" y2="10.16" width="0.8128" layer="16"/>
+<wire x1="30.226" y1="10.16" x2="27.178" y2="13.208" width="0.8128" layer="16"/>
+<wire x1="27.178" y1="13.208" x2="27.178" y2="16.256" width="0.8128" layer="16"/>
+<via x="27.178" y="16.256" extent="1-16" drill="0.6"/>
+<wire x1="27.178" y1="16.256" x2="27.178" y2="16.4592" width="0.6096" layer="1"/>
+<wire x1="27.178" y1="16.4592" x2="26.5176" y2="17.1196" width="0.6096" layer="1"/>
+<wire x1="49.3776" y1="10.16" x2="49.3776" y2="12.7" width="0.8128" layer="16"/>
+<wire x1="49.3776" y1="7.62" x2="49.3776" y2="10.16" width="0.8128" layer="16"/>
 </signal>
 <signal name="N$3">
