File: Circuit/P1R4/CD.sch (EAGLE design)
At the start: 126 parts, among them U1 MK20DX256VLH7, U2 TPS61200, U3 MPU-9250, Y1 32.768KHz, Y2 16Mhz/8pF, Y3 26 Mhz, Y4 16 Mhz

Commit message: Fixed Wifi wiring, mild rearranging of IO. Pinout documented on Google. Antennae isolated and via fenced
Parts:
- added R51: 10k, SparkFun-Resistors:RESISTOR0603-RES
Connections:
- removed net N$9: R17.1, U1.PTC3
- new net N$8: R51.2, U$6.MTDO/13
- new net PTC3: U$6.XPD_DCDC/8, U1.PTC3
- net GND: now also R51.1
- net PTB16: now also U$6.U0TXD/26; no longer U$6.U0RXD/25
- net PTB17: now also U$6.U0RXD/25; no longer U$6.U0TXD/26
- net PTD7: now also R17.1
Other:
- moved on the sheet: C10, C12, C13, C14, C15, C24, C25, C27, C36, C37, C8, C9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

Commit message: Preliminary Final R4 finished
Connections:
- net N$8 renamed MTDO
Changed lines of the file:
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@@
 <setting verticaltext="up"/>
 </settings>
-<grid distance="0.05" unitdist="inch" unit="inch" style="lines" multiple="1" display="no" altdistance="0.01" altunitdist="inch" altunit="inch"/>
+<grid distance="0.1" unitdist="inch" unit="inch" style="lines" multiple="1" display="no" altdistance="0.01" altunitdist="inch" altunit="inch"/>
 <layers>
 <layer number="1" name="Top" color="4" fill="1" visible="no" active="no"/>
@@
 </segment>
 </net>
-<net name="N$8" class="0">
+<net name="MTDO" class="0">
 <segment>
 <pinref part="U$6" gate="G$1" pin="MTDO/13"/>
