File: Circuit/P1R4/final/CD.sch (EAGLE design)
At the start: 65 parts, among them U1 MK20DX256VLH7, U2 TPS61200, U3 MPU-9250, Y1 32.768KHz, Y2 16Mhz/8pF, Y3 26 Mhz, Y4 16 Mhz

Commit message: Cleaned and organized circuit design directories
Parts:
- removed JP2, JP3, JP4: (no value), SparkFun-Connectors:M08SILK_FEMALE_PTH
- removed JP6: M100.1, umich:M100.1
- added C26, C28, C33, C34, C35, C36, C37: .1 uF, SparkFun-Capacitors:CAP0603-CAP
- added C29, C30, C31, C32: 22 pF, appfruits:CAPACITOR-10UF
- added JP1: (no value), SparkFun-Connectors:M15
- added L7, L8: (no value), SparkFun-Passives:INDUCTOR30OHM,1.8A
- added LED2, LED4: (no value), appfruits:LED-GREEN
- added R15: 12k, SparkFun-Resistors:RESISTOR0603-RES
- added R17, R8: 330, appfruits:RESISTOR-470
- added R18: 200, SparkFun-Resistors:RESISTOR0603-RES
- added R19, R20, R21, R22, R23, R24: 10k, SparkFun:RESISTOR0603-RES
- added R25, R26, R27, R28, R29, R30, R31, R32, R33, R34, R35, R36, R37, R38, R39, R40, R41, R42, R43, R44, R45, R46, R47, R48, R49, R50, R52, R53: (no value), SparkFun:RESISTOR0402-RES
- added R51: 10k, SparkFun-Resistors:RESISTOR0603-RES
- added U$11, U$13, U$14, U$15, U$16, U$17, U$18, U$8: LTST-C19FD1WT, led:LTST-C19FD1WT
- added U$20, U$21: PCA9552BS, NXP_By_element14_Batch_1:PCA9552BS
- added U$7: 2X5_0.05"_CORTEX_DEBUGTH_NOKEY_UNSHROUDED, con-cortex:2X5_0.05"_CORTEX_DEBUGTH_NOKEY_UNSHROUDED
Connections:
- removed net ID: JP6.6, U1.PTA1
- removed net N$30: U1.EXTAL32, Y1.1
- removed net PTB2: U1.PTB2
- removed net PTB3: U1.PTB3
- removed net PTC2: U1.PTC2
- removed net SWD_CLK: JP6.4, U1.PTA0
- removed net SWD_DIO: JP6.5, U1.PTA3
- removed net VDD: R13.1, R14.1, U$6.VDDA/30
- new net AD0: U1.PTC2, U3.AD0/MISO
- new net MTDO: R51.2, U$6.MTDO/13
- new net N$10: C31.2, U1.XTAL32, Y1.2
- new net N$100: R39.2, U$15.G
- new net N$101: R43.1, U$21.LED8
- new net N$102: R47.1, U$21.LED9
- new net N$103: R48.1, U$21.LED10
- new net N$104: R46.1, U$21.LED11
- new net N$105: U$21.LED12
- new net N$106: R24.1, U$21.A2
- new net N$107: R23.1, U$21.A1
- new net N$108: R22.1, U$21.A0
- new net N$109: R40.2, U$16.B
- new net N$11: C32.2, U1.EXTAL32, Y1.1
- new net N$112: R41.2, U$16.R
- new net N$113: R42.2, U$16.G
- new net N$114: R43.2, U$17.B
- new net N$115: R44.2, U$17.R
- new net N$116: R45.2, U$17.G
- new net N$117: R46.2, U$18.B
- new net N$118: R47.2, U$18.R
- new net N$119: R48.2, U$18.G
- new net N$35: R18.1, U$3.CLK
- new net N$39: R26.2, U$8.R
- new net N$40: R19.1, U$20.A2
- new net N$41: R27.2, U$8.B
- new net N$42: R25.2, U$8.G
- new net N$45: R28.2, U$11.B
- new net N$46: R29.2, U$11.R
- new net N$47: R30.2, U$11.G
- new net N$48: R27.1, U$20.LED2
- new net N$49: R26.1, U$20.LED0
- new net N$50: R31.2, U$13.B
- new net N$51: R28.1, U$20.LED5
- new net N$60: R32.2, U$13.R
- new net N$61: R33.2, U$13.G
- new net N$62: R34.2, U$14.B
- new net N$63: R35.2, U$14.R
- new net N$7: LED2.A, R8.2
- new net N$73: R25.1, U$20.LED1
- new net N$75: R29.1, U$20.LED3
- new net N$76: R30.1, U$20.LED4
- new net N$78: R32.1, U$20.LED6
- new net N$79: R33.1, U$20.LED7
- new net N$80: R31.1, U$20.LED8
- new net N$81: R36.2, U$14.G
- new net N$82: R35.1, U$20.LED9
- new net N$83: R36.1, U$20.LED10
- new net N$84: R34.1, U$20.LED11
- new net N$85: U$20.LED12
- new net N$86: R37.2, U$15.B
- new net N$87: R20.1, U$20.A1
- new net N$88: R21.1, U$20.A0
- new net N$89: R38.2, U$15.R
- new net N$92: R38.1, U$21.LED0
- new net N$93: R39.1, U$21.LED1
- new net N$94: R37.1, U$21.LED2
- new net N$95: R41.1, U$21.LED3
- new net N$96: R42.1, U$21.LED4
- new net N$97: R40.1, U$21.LED5
- new net N$98: R44.1, U$21.LED6
- new net N$99: R45.1, U$21.LED7
- new net PTA0: R50.2, U$7.SWDCLK/TCK, U1.PTA0
- new net PTA1: R52.2, U$7.NC/TDI, U1.PTA1
- new net PTA3: R49.2, U$7.SWDIO/TMS, U1.PTA3
- net 3.3V: now also C26.2, C28.2, C33.1, C34.1, C35.1, C36.1, C37.2, JP1.13, JP1.14, JP1.15, R13.1, R14.1, R15.2, R22.2, R49.1, R52.1, R53.1, R9.1, U$11.V, U$13.V, U$14.V, U$15.V, U$16.V, U$17.V, U$18.V, U$20.VDD, U$21.VDD, U$4.VDD/15, U$6.VDDA/30, U$7.VCC, U$8.V; no longer JP4.1, JP4.2, JP4.3, JP4.4, JP4.5, JP4.6, JP4.7, JP4.8, JP6.1, LED1.A
- net GND: now also C26.1, C28.1, C29.1, C30.1, C31.1, C32.1, C33.2, C34.2, C35.2, C36.2, C37.1, JP1.1, JP1.2, JP1.3, JP1.4, L7.2, L8.2, LED1.C, LED2.C, LED4.C, R19.2, R20.2, R21.2, R23.2, R24.2, R50.1, R51.1, U$20.VSS, U$21.VSS, U$4.VSS/14, U$7.GND, U$7.GND-DETECT; no longer JP3.1, JP3.2, JP3.3, JP3.4, JP3.5, JP3.6, JP3.7, JP3.8, JP6.10, R9.2
- net N$1: now also LED1.A, R9.2; no longer LED1.C, R9.1
- net N$13: now also L8.1
- net N$16: now also L7.1
- net N$20: no longer U$4.VDD/15, U$4.VSS/14
- net N$27: now also C29.2
- net N$28: now also C30.2
- net N$29: now also LED4.A, R17.2; no longer U1.XTAL32, Y1.2
- net PTA2: now also U$7.SWO/TDO; no longer JP6.3
- net PTB16: now also U$6.U0TXD/26; no longer U$6.U0RXD/25
- net PTB17: now also U$6.U0RXD/25; no longer U$6.U0TXD/26
- net PTC0: now also R15.1
- net PTC10: now also JP1.12
- net PTC11: now also JP1.11
- net PTC3: now also U$6.XPD_DCDC/8
- net PTD0: now also JP1.10
- net PTD1: now also JP1.9
- net PTD2: now also JP1.8
- net PTD3: now also JP1.7
- net PTD4: now also JP1.6
- net PTD5: now also JP1.5
- net PTD6: now also R8.1
- net PTD7: now also R17.1
- net RESET_B: now also R53.2, U$7.~RESET; no longer JP6.2
- net SCL: now also U$20.SCL, U$21.SCL, U1.PTB2
- net SD-CLK: now also R18.2; no longer U$3.CLK
- net SDA: now also U$20.SDA, U$21.SDA, U1.PTB3
- net USB_D_N: no longer JP6.8
- net USB_D_P: no longer JP6.7
- net VCC: no longer JP6.9
Other:
- note added: "3.3V Breakout"
- note added: "Connections for JTAG/USB+Bootloader"
- note added: "I2C power"
- note added: "RESET to PTC0 active low therefore pulled up"
- note added: "RTC"
- note added: "SCL"
- note added: "SDA"
- note added: "Switch for VRAW (raw voltage from Lipo) to VCC into regulator"
- note removed: "If you don't want to waste energy remove this power led as all it does is indicating applied power."
- note removed: "Parts of this these schematics were inspired/taken from Teensy 3.1 schematics published by Paul J. Stoffregen at www.pjrc.com and Sparkfuns Power Cell schematics (https://www.sparkfun.com/products/11231) These schematics have been successfully working in a real world project and are provided as a reference for your own custom board."
- note removed: "Published June 2015 by Phillip Schuster (www.appfruits.com)"
- note removed: "Released under the Creative Commons Attribution Share-Alike 4.0 License https://creativecommons.org/licenses/by-sa/4.0/"
