File: Circuit/P1R4/final/P1R4.sch (EAGLE design)
At the start: 129 parts, among them J1 MICRO_USB_B_HIROSE_ZX62R-B-5P, U1 MK20DX256VLH7, U2 TPS61200, U3 MPU-9250, Y1 32.768KHz, Y2 16Mhz/8pF, Y3 26 Mhz, Y4 16 Mhz

Commit message: Added four from LED drivers to R4. Corrected R3 bootloader circuit. Rerouted switch in schematic and board on both R3 and R4 for proper isolation of USB and lipo voltage. Ready for final review
Parts:
- removed J1: MICRO_USB_B_HIROSE_ZX62R-B-5P, connector:MICRO_USB_B_HIROSE_ZX62R-B-5P
- removed U$22: MINI54TAN, TeensyCustom:MINI54TAN
- added JP2: (no value), SparkFun-Connectors:M04LOCK
Connections:
- new net N$8: JP2.3, U$20.LED13
- new net N$9: U$21.LED14
- new net N$90: U$21.LED15
- new net N$91: JP2.2, U$20.LED14
- net N$105: now also JP2.1, U$20.LED15; no longer U$21.LED12
- net N$85: now also JP2.4
- net VCC: now also S1.P; no longer S1.O
- net VRAW: now also S1.O; no longer S1.P
Other:
- moved on the sheet: S1
Changed lines of the file:
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@@
 <part name="R51" library="SparkFun-Resistors" deviceset="RESISTOR" device="0603-RES" value="10k"/>
 <part name="GND17" library="SparkFun" deviceset="GND" device=""/>
-<part name="U$22" library="TeensyCustom" deviceset="MINI54TAN" device=""/>
-<part name="J1" library="connector" deviceset="MICRO_USB_B_HIROSE_ZX62R-B-5P" device=""/>
+<part name="JP2" library="SparkFun-Connectors" deviceset="M04" device="LOCK"/>
 </parts>
 <sheets>
@@
 <instance part="GND1" gate="1" x="226.06" y="-22.86"/>
 <instance part="JP5" gate="G$1" x="17.78" y="-17.78"/>
-<instance part="S1" gate="1" x="33.02" y="-15.24"/>
+<instance part="S1" gate="1" x="38.1" y="-17.78" rot="R180"/>
 <instance part="R8" gate="G$1" x="254" y="-60.96"/>
 <instance part="LED2" gate="G$1" x="264.16" y="-60.96" rot="R90"/>
@@
 <instance part="R52" gate="G$1" x="111.76" y="-170.18" rot="R180"/>
 <instance part="R53" gate="G$1" x="111.76" y="-167.64" rot="R180"/>
-<instance part="U$22" gate="G$1" x="43.18" y="-152.4"/>
-<instance part="J1" gate="G$1" x="30.48" y="-114.3" rot="R180"/>
 </instances>
 <busses>
@@
 </segment>
 <segment>
-<pinref part="S1" gate="1" pin="O"/>
-<wire x1="38.1" y1="-12.7" x2="40.64" y2="-12.7" width="0.1524" layer="91"/>
+<pinref part="S1" gate="1" pin="P"/>
+<wire x1="40.64" y1="-17.78" x2="43.18" y2="-17.78" width="0.1524" layer="91"/>
 </segment>
 </net>
@@
 </segment>
 </net>
-<net name="VRAW" class="2">
-<segment>
-<pinref part="JP5" gate="G$1" pin="2"/>
-<pinref part="S1" gate="1" pin="P"/>
-<wire x1="25.4" y1="-15.24" x2="30.48" y2="-15.24" width="0.1524" layer="91"/>
-</segment>
-</net>
 <net name="PTC8" class="0">
 <segment>
@@
 <pinref part="U1" gate="G$1" pin="PTC3"/>
 <wire x1="203.2" y1="-91.44" x2="210.82" y2="-91.44" width="0.1524" layer="91"/>
+</segment>
+</net>
+<net name="VRAW" class="0">
+<segment>
+<pinref part="S1" gate="1" pin="O"/>
+<wire x1="33.02" y1="-20.32" x2="30.48" y2="-20.32" width="0.1524" layer="91"/>
+<pinref part="JP5" gate="G$1" pin="2"/>
+<wire x1="25.4" y1="-15.24" x2="30.48" y2="-15.24" width="0.1524" layer="91"/>
+<wire x1="30.48" y1="-15.24" x2="30.48" y2="-20.32" width="0.1524" layer="91"/>
 </segment>
 </net>
@@
 <instance part="R47" gate="G$1" x="93.98" y="27.94" rot="R90"/>
 <instance part="R48" gate="G$1" x="99.06" y="27.94" rot="R90"/>
+<instance part="JP2" gate="G$1" x="-7.62" y="-73.66" rot="R180"/>
 </instances>
 <busses>
@@
 <pinref part="U$20" gate="G$1" pin="LED12"/>
 <wire x1="-38.1" y1="-81.28" x2="-35.56" y2="-81.28" width="0.1524" layer="91"/>
+<wire x1="-35.56" y1="-81.28" x2="-35.56" y2="-78.74" width="0.1524" layer="91"/>
+<pinref part="JP2" gate="G$1" pin="4"/>
+<wire x1="-35.56" y1="-78.74" x2="-12.7" y2="-78.74" width="0.1524" layer="91"/>
 </segment>
 </net>
@@
 <pinref part="R46" gate="G$1" pin="1"/>
 <wire x1="88.9" y1="15.24" x2="88.9" y2="22.86" width="0.1524" layer="91"/>
-</segment>
-</net>
-<net name="N$105" class="0">
-<segment>
-<pinref part="U$21" gate="G$1" pin="LED12"/>
-<wire x1="86.36" y1="-83.82" x2="88.9" y2="-83.82" width="0.1524" layer="91"/>
 </segment>
 </net>
@@
 </segment>
 </net>
+<net name="N$9" class="0">
+<segment>
+<pinref part="U$21" gate="G$1" pin="LED14"/>
+<wire x1="86.36" y1="-73.66" x2="129.54" y2="-73.66" width="0.1524" layer="91"/>
+<wire x1="129.54" y1="-73.66" x2="129.54" y2="-76.2" width="0.1524" layer="91"/>
+</segment>
+</net>
+<net name="N$90" class="0">
+<segment>
+<pinref part="U$21" gate="G$1" pin="LED15"/>
+<wire x1="86.36" y1="-68.58" x2="139.7" y2="-68.58" width="0.1524" layer="91"/>
+</segment>
+</net>
+<net name="N$8" class="0">
+<segment>
+<pinref part="U$20" gate="G$1" pin="LED13"/>
+<pinref part="JP2" gate="G$1" pin="3"/>
+<wire x1="-38.1" y1="-76.2" x2="-12.7" y2="-76.2" width="0.1524" layer="91"/>
+</segment>
+</net>
+<net name="N$91" class="0">
+<segment>
+<pinref part="U$20" gate="G$1" pin="LED14"/>
+<wire x1="-38.1" y1="-71.12" x2="-38.1" y2="-73.66" width="0.1524" layer="91"/>
+<pinref part="JP2" gate="G$1" pin="2"/>
+<wire x1="-38.1" y1="-73.66" x2="-12.7" y2="-73.66" width="0.1524" layer="91"/>
+</segment>
+</net>
+<net name="N$105" class="0">
+<segment>
+<pinref part="U$20" gate="G$1" pin="LED15"/>
+<wire x1="-38.1" y1="-66.04" x2="-35.56" y2="-66.04" width="0.1524" layer="91"/>
+<wire x1="-35.56" y1="-66.04" x2="-35.56" y2="-71.12" width="0.1524" layer="91"/>
+<pinref part="JP2" gate="G$1" pin="1"/>
+<wire x1="-35.56" y1="-71.12" x2="-12.7" y2="-71.12" width="0.1524" layer="91"/>
+</segment>
+</net>

Commit message: R3 and R4 DRC checked and ready for final review
Parts:
- removed JP2: (no value), SparkFun-Connectors:M04LOCK
- added JP3: (no value), SparkFun:M04PTH
Connections:
- net N$105: now also JP3.1; no longer JP2.1
- net N$8: now also JP3.3; no longer JP2.3
- net N$85: now also JP3.4; no longer JP2.4
- net N$91: now also JP3.2; no longer JP2.2
Changed lines of the file:
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@@
 <part name="R51" library="SparkFun-Resistors" deviceset="RESISTOR" device="0603-RES" value="10k"/>
 <part name="GND17" library="SparkFun" deviceset="GND" device=""/>
-<part name="JP2" library="SparkFun-Connectors" deviceset="M04" device="LOCK"/>
+<part name="JP3" library="SparkFun" deviceset="M04" device="PTH"/>
 </parts>
 <sheets>
@@
 <instance part="R47" gate="G$1" x="93.98" y="27.94" rot="R90"/>
 <instance part="R48" gate="G$1" x="99.06" y="27.94" rot="R90"/>
-<instance part="JP2" gate="G$1" x="-7.62" y="-73.66" rot="R180"/>
+<instance part="JP3" gate="G$1" x="-10.16" y="-73.66" rot="R180"/>
 </instances>
 <busses>
@@
 <wire x1="-38.1" y1="-81.28" x2="-35.56" y2="-81.28" width="0.1524" layer="91"/>
 <wire x1="-35.56" y1="-81.28" x2="-35.56" y2="-78.74" width="0.1524" layer="91"/>
-<pinref part="JP2" gate="G$1" pin="4"/>
-<wire x1="-35.56" y1="-78.74" x2="-12.7" y2="-78.74" width="0.1524" layer="91"/>
+<pinref part="JP3" gate="G$1" pin="4"/>
+<wire x1="-35.56" y1="-78.74" x2="-15.24" y2="-78.74" width="0.1524" layer="91"/>
 </segment>
 </net>
@@
 </segment>
 </net>
-<net name="N$8" class="0">
-<segment>
-<pinref part="U$20" gate="G$1" pin="LED13"/>
-<pinref part="JP2" gate="G$1" pin="3"/>
-<wire x1="-38.1" y1="-76.2" x2="-12.7" y2="-76.2" width="0.1524" layer="91"/>
-</segment>
-</net>
 <net name="N$91" class="0">
 <segment>
 <pinref part="U$20" gate="G$1" pin="LED14"/>
 <wire x1="-38.1" y1="-71.12" x2="-38.1" y2="-73.66" width="0.1524" layer="91"/>
-<pinref part="JP2" gate="G$1" pin="2"/>
-<wire x1="-38.1" y1="-73.66" x2="-12.7" y2="-73.66" width="0.1524" layer="91"/>
+<pinref part="JP3" gate="G$1" pin="2"/>
+<wire x1="-38.1" y1="-73.66" x2="-15.24" y2="-73.66" width="0.1524" layer="91"/>
 </segment>
 </net>
@@
 <wire x1="-38.1" y1="-66.04" x2="-35.56" y2="-66.04" width="0.1524" layer="91"/>
 <wire x1="-35.56" y1="-66.04" x2="-35.56" y2="-71.12" width="0.1524" layer="91"/>
-<pinref part="JP2" gate="G$1" pin="1"/>
-<wire x1="-35.56" y1="-71.12" x2="-12.7" y2="-71.12" width="0.1524" layer="91"/>
-</segment>
-</net>
+<pinref part="JP3" gate="G$1" pin="1"/>
+<wire x1="-35.56" y1="-71.12" x2="-15.24" y2="-71.12" width="0.1524" layer="91"/>
+</segment>
+</net>
+<net name="N$8" class="0">
+<segment>
+<pinref part="U$20" gate="G$1" pin="LED13"/>
+<pinref part="JP3" gate="G$1" pin="3"/>
+<wire x1="-38.1" y1="-76.2" x2="-15.24" y2="-76.2" width="0.1524" layer="91"/>
+</segment>
+</net>

Commit message: Added some part names to P1R4 to make assembly suck less
Other:
- note added: "U20"
- note added: "U21"
- note added: "U3"
- note added: "U4"
- note added: "U5"
- note added: "U6"
Changed lines of the file:
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@@
 active low
 therefore pulled up</text>
+<text x="-12.7" y="81.28" size="1.778" layer="91">U6</text>
+<text x="33.02" y="68.58" size="1.778" layer="91">U3</text>
+<text x="86.36" y="66.04" size="1.778" layer="91">U4</text>
+<text x="208.28" y="66.04" size="1.778" layer="91">U5</text>
 </plain>
 <instances>
@@
 <text x="-50.8" y="-39.37" size="1.778" layer="91">SCL</text>
 <text x="72.39" y="-45.72" size="1.778" layer="91">SCL</text>
+<text x="-45.72" y="-48.26" size="1.778" layer="91">U20</text>
+<text x="83.82" y="-53.34" size="1.778" layer="91">U21</text>
 </plain>
 <instances>
