File: Circuit/P1R5/P1R5.sch (EAGLE design)
At the start: 30 parts, among them U1 MK20DX256VLH7, Y1 32.768KHz, Y2 16Mhz/8pF

Commit message: more cleanup on micro.
Connections:
- removed net PTC10: JP1.12, U1.PTC10
- removed net PTC11: JP1.11, U1.PTC11
- removed net PTD0: JP1.10, U1.PTD0
- removed net PTD1: JP1.9, U1.PTD1
- removed net PTD2: JP1.8, U1.PTD2
- removed net PTD3: JP1.7, U1.PTD3
- removed net PTD4: JP1.6, U1.PTD4
- removed net PTD5: JP1.5, U1.PTD5
- removed net PTD6: R8.1, U1.PTD6
- removed net PTD7: R17.1, U1.PTD7
- new net N$10: LED2.C, U1.PTD6
- new net N$13: LED4.C, U1.PTD7
- new net N$16: JP1.11, U1.PTC11/I2C1_SDA
- new net N$17: JP1.10, U1.PTD0/SPI0_PCS0
- new net N$18: JP1.9, U1.PTD1/SPI0_SCK
- new net N$19: JP1.8, U1.PTD2/SPI0_SOUT
- new net N$20: JP1.7, U1.PTD3/SPI0_SIN
- new net N$21: JP1.6, U1.PTD4/SPI0_PCS1
- new net N$23: JP1.5, U1.PTD5/SPI0_PCS2
- new net N$24: JP1.12, U1.PTC10/I2C1_SCL
- net 3.3V: now also R17.1, R8.1
- net GND: no longer LED2.C, LED4.C
- net N$8: now also U1.PTA18/EXTAL0; no longer U1.PTA18
- net N$9: now also U1.PTA19/XTAL0; no longer U1.PTA19
- net PTA0: now also U1.PTA0/TCLK; no longer U1.PTA0
- net PTA1: now also U1.PTA1/TDI; no longer U1.PTA1
- net PTA2: now also U1.PTA2/TDO; no longer U1.PTA2
- net PTA3: now also U1.PTA3/TMS; no longer U1.PTA3
Other:
- note removed: "3.3V Breakout"
- moved on the sheet: JP1, LED2, LED4, R17, R8, U1

Commit message: hierarchical blocks done.
Parts:
- added R13, R14: 10k, SparkFun-Resistors:RESISTOR0603-RES
Connections:
- net PTB0 renamed N$27
- net PTB1 renamed N$28
- net PTB16 renamed N$34
- net PTB17 renamed N$35
- net PTB18 renamed N$38
- net PTB19 renamed N$39
- net PTC1 renamed N$41
- net PTC3 renamed N$40
- net PTC4 renamed N$46
- net PTC5 renamed N$47
- net PTC6 renamed N$48
- net PTC7 renamed N$49
- net PTC8 renamed N$42
- net PTC9 renamed N$45
- removed net A12: U1.ADC0_DP3
- removed net A13: U1.ADC0_DM3
- removed net AD0: U1.PTC2
- removed net DAC/A14: U1.DAC0
- removed net PTA12: U1.PTA12
- removed net PTA13: U1.PTA13
- removed net PTA4: U1.PTA4
- removed net PTA5: U1.PTA5
- removed net PTC0: U1.PTC0
- removed net PTE0: U1.PTE0
- removed net PTE1: U1.PTE1
- removed net SCL: U1.PTB2
- removed net SDA: U1.PTB3
- removed net USB_D_N: U1.USB0_DM
- removed net USB_D_P: U1.USB0_DP
- new net N$25: R14.2, U1.PTB2
- new net N$26: R13.2, U1.PTB3
- net 3.3V: now also R13.1, R14.1
Other:
- note removed: "I2C power"
- moved on the sheet: JP1, JP5, S1

Commit message: labels made on all hierarchical blocks and nets
pretty much all connected back up. Not sure it's showing through on the
schematic yet.
Connections:
- net N$19 renamed 
- net N$25 renamed SCL
- net N$26 renamed SDA
- net N$27 renamed INT
- net N$28 renamed FSYNC
- net N$32 renamed V_IN
- net N$34 renamed U0TX
- net N$35 renamed U0RX
- net N$38 renamed GPIO0
- net N$39 renamed GPIO2
- net N$40 renamed XPD_DCDC
- net N$41 renamed CHIP_EN
- net N$42 renamed IRQ
- net N$45 renamed CE
- net N$46 renamed CSN
- net N$47 renamed SCK
- net N$48 renamed MOSI
- net N$49 renamed MISO
- new net WIFI_RESET: U1.PTC0
Other:
- note removed: "RESET to PTC0 active low therefore pulled up"
- note removed: "SCL"
- note removed: "SDA"
- note removed: "Source"

Commit message: moved libraries, regenerated PCB, reannotated design, connected hierarchical blocks.
Parts:
- removed C16, C18, C19, C21: 0.1uF, appfruits:CAPACITOR-0.1UF
- removed C17, C20: 2.2uF, appfruits:CAPACITOR-2.2UF
- removed C29, C30, C31, C32: 10uF, appfruits:CAPACITOR-10UF
- removed JP5: (no value), SparkFun-Connectors:M02PTH
- removed L3, L4: 600 Ohm/100 Mhz, appfruits:INDUCTOR-BK2125HM601-T
- removed LED4: (no value), appfruits:LED-GREEN
- removed R13, R14: 10k, SparkFun-Resistors:RESISTOR0603-RES
- removed R16, R17: 470, appfruits:RESISTOR-470
- removed R50, R52, R53: (no value), SparkFun:RESISTOR0402-RES
- added C1, C7: 2.2uF, appfruits:CAPACITOR-2.2UF
- added C10, C12, C9: 10uF, appfruits:CAPACITOR-10UF
- added C2, C3, C4, C6, C8: 0.1uF, appfruits:CAPACITOR-0.1UF
- added JP2: (no value), SparkFun-Connectors:M15
- added L1, L2: 600 Ohm/100 Mhz, appfruits:INDUCTOR-BK2125HM601-T
- added LED1: (no value), appfruits:LED-GREEN
- added R1, R6, R7: 470, appfruits:RESISTOR-470
- added R3, R4, R5: (no value), SparkFun:RESISTOR0402-RES
- added R9: 10k, SparkFun-Resistors:RESISTOR0603-RES
- C11: value 0.1uF -> 10uF; device appfruits:CAPACITOR-0.1UF -> appfruits:CAPACITOR-10UF
- JP1: device SparkFun-Connectors:M15 -> SparkFun-Connectors:M02PTH
- R8: value 470 -> 10k; device appfruits:RESISTOR-470 -> SparkFun-Resistors:RESISTOR0603-RES
- Y1: value 32.768KHz -> 16Mhz/8pF; device appfruits:CRYSTAL/32.768KHZ/SMD-TXC_7A -> appfruits:CRYSTAL/SMD-5X3-GND16MHZ/8PF; MF Epson Timing -> ECS; MPN FC-255 32.7680K-A3 -> ECS-160-8-30B-CKM
- Y2: value 16Mhz/8pF -> 32.768KHz; device appfruits:CRYSTAL/SMD-5X3-GND16MHZ/8PF -> appfruits:CRYSTAL/32.768KHZ/SMD-TXC_7A; MF ECS -> Epson Timing; MPN ECS-160-8-30B-CKM -> FC-255 32.7680K-A3
- renumbered R49 to R2, U$7 to J1
Connections:
- removed net : JP1.8, U1.PTD2/SPI0_SOUT
- removed net SCL: R14.2, U1.PTB2
- new net CHANGE: JP2.8, U1.PTD2/SPI0_SOUT
- new net N$12: C8.2
- new net N$14: C12.1, C6.1
- new net N$3: C2.2, R3.1, R4.2, U1.PTC2
- new net N$4: R6.2, R7.1, R8.2, U1.PTB2
- new net N$5: LED1.A, R9.2
- new net V_OUT: C3.1, R7.2, R9.1
- net 3.3V: now also C2.1, C3.1, C4.1, C5.1, C7.1, JP2.13, JP2.14, JP2.15, L1.2, R4.1, R5.1, R6.1, R7.1, R9.1; no longer C19.1, C20.1, JP1.13, JP1.14, JP1.15, L3.2, R13.1, R14.1, R17.1, R52.1, R53.1
- net GND: now also C1.2, C10.1, C10.2, C11.1, C12.1, C12.2, C2.2, C3.2, C4.2, C7.2, C8.1, C9.1, C9.2, JP2.1, JP2.2, JP2.3, JP2.4, L2.1, LED1.C, R1.2, R3.1, R4.1, R5.1, R6.1; no longer C18.2, C19.2, C20.2, C21.2, C29.1, C30.1, C31.1, C32.1, JP1.1, JP1.3, JP1.4, L4.1, R50.1
- net N$1: now also C10.1, C11.2, C9.1, L1.1, L2.2, Y2.2; no longer C31.2, Y1.2
- net N$10: now also LED1.C; no longer LED2.C
- net N$11: now also C7.1; no longer C18.1, C21.1, C5.1
- net N$110: now also JP1.1; no longer JP5.1
- net N$13: now also L2.1, LED2.C; no longer LED4.C
- net N$16: now also JP2.11, R5.2; no longer JP1.11
- net N$17: now also JP2.10; no longer JP1.10
- net N$18: now also JP2.9; no longer JP1.9
- net N$2: now also C12.2, C4.1, Y2.1; no longer C32.2, Y1.1
- net N$20: now also JP2.7; no longer JP1.7
- net N$21: now also JP2.6; no longer JP1.6
- net N$23: now also JP2.5; no longer JP1.5
- net N$24: now also JP2.12; no longer JP1.12
- net N$29: now also LED2.A, R7.2; no longer LED4.A, R17.2
- net N$7: now also C6.2, LED1.A, R6.2; no longer LED2.A, R8.2
- net N$8: now also C9.2, R1.1, Y1G$1.2; no longer C29.2, Y2G$1.2
- net N$9: now also C10.2, Y1G$1.1; no longer C30.2, Y2G$1.1
- net PTA0: now also R3.2; no longer R50.2
- net PTA1: now also R4.2; no longer R52.2
- net RESET_B: now also R5.2; no longer R53.2
- net SDA: now also R9.2; no longer R13.2
- net VDDA: now also C1.1, L1.1, R1.1; no longer C17.1, L3.1, R16.1
- net VREFH: now also C6.1, R1.2; no longer C11.1, R16.2
- net VREFL: now also C1.2, C6.2, C8.2, L2.2; no longer C11.2, C16.2, C17.2, L4.2
- net VREF_OUT: now also C8.1; no longer C16.1
- net V_IN: now also C1.1, C2.1, L1.2, R3.2
Other:
- note added: "Switch for VIN from LiPO to VCC into regulator"
- note removed: "Switch for VRAW (raw voltage from Lipo) to VCC into regulator"
- moved on the sheet: C11, C5, LED2, R8, Y1G$1, Y2

Commit message: notes
Added orientation note to IMU
Added placement notes to gpio blocks and replaced header with test
points.
Verified IMU and WiFi modules
Parts:
- removed JP2: (no value), SparkFun-Connectors:M15
- added TP1, TP10, TP11, TP12, TP13, TP14, TP15, TP16, TP17, TP18, TP19, TP2, TP20, TP21, TP22, TP23, TP24, TP25, TP26, TP27, TP28, TP29, TP3, TP30, TP31, TP32, TP33, TP34, TP35, TP36, TP4, TP5, TP6, TP7, TP8, TP9: TPPAD1-20, testpad:TPPAD1-20
Connections:
- removed net CHANGE: JP2.8, U1.PTD2/SPI0_SOUT
- removed net N$23: JP2.5, U1.PTD5/SPI0_PCS2
- removed net N$24: JP2.12, U1.PTC10/I2C1_SCL
- new net N$15: TP10.TP, U1.PTD0/SPI0_PCS0
- new net N$19: TP14.TP, U1.PTE1/I2C1_SCL/UART1_RX
- new net N$6: TP8.TP, U1.PTD2/SPI0_SOUT
- new net VCC: C1.1, C2.1, C5.1, C7.1
- net 3.3V: now also TP17.TP, TP18.TP, TP22.TP, TP23.TP, TP24.TP, TP28.TP, TP29.TP, TP30.TP, TP34.TP, TP35.TP, TP36.TP, TP4.TP; no longer JP2.13, JP2.14, JP2.15
- net GND: now also TP1.TP, TP19.TP, TP2.TP, TP20.TP, TP21.TP, TP25.TP, TP26.TP, TP27.TP, TP3.TP, TP31.TP, TP32.TP, TP33.TP; no longer JP2.1, JP2.2, JP2.3, JP2.4
- net N$11: now also TP9.TP, U1.PTD1/SPI0_SCK
- net N$12: now also TP5.TP, U1.PTD5/SPI0_PCS2
- net N$14: now also TP6.TP, U1.PTD4/SPI0_PCS1
- net N$16: now also TP11.TP; no longer JP2.11
- net N$17: now also TP12.TP, U1.PTC10/I2C1_SCL; no longer JP2.10, U1.PTD0/SPI0_PCS0
- net N$18: now also TP13.TP, U1.PTE0/I2C1_SDA/UART1_TX; no longer JP2.9, U1.PTD1/SPI0_SCK
- net N$20: now also TP15.TP, U1.PTA13/CAN0_RX; no longer JP2.7, U1.PTD3/SPI0_SIN
- net N$21: now also TP16.TP, U1.PTA12/CAN0_TX; no longer JP2.6, U1.PTD4/SPI0_PCS1
- net N$5: now also TP7.TP, U1.PTD3/SPI0_SIN
Other:
- note added: "+X Accelerometer +Y Compass"
- note added: "+Y Accelerometer +X Compass"
- note added: "FIX THIS PINOUT"
- note added: "I/O Groups"
- note added: "I/O Groups: Place at board edge as noted by group name. Place the I/O towards the inside. Place ground at the board edge. Place power in between."
- note added: "I2C Address: 1100<A2><A1><A0>"
- note added: "I2C Address: 110100X X = AD0"
- note added: "Orient X and Y of Accelerometer along with PCB."
- note added: "Place decoupling caps near VDD pins on drivers"
- note added: "X+ Group"
- note added: "X- Group"
- note added: "Y+ Group"
- note added: "Y- Group"
- note removed: "Connections for JTAG/USB+Bootloader"
- moved on the sheet: U1

Commit message: More schematic cleanup.
Verified layouts, will probably check them again anyway.
Still need to do the passives and fix part numbers so they match the
bom-ex db.
Parts:
- added AE1, AE2: ANTENNA2SMD, SparkFun-RF:ANTENNA2SMD
- added C13, C15, C17, C19, C36: 0.1uF, appfruits:CAPACITOR-0.1UF
- added C14: 10uF, appfruits:CAPACITOR-10UF
- added C16: 22uF, appfruits:CAPACITOR-22UF
- added C18, C20, C37: 2.2uF, appfruits:CAPACITOR-2.2UF
- added C21, C22, C23, C24, C25, C28, C31, C32, C34, C35: .1 uF, SparkFun-Capacitors:CAP0603-CAP
- added C26, C27: 15 pF, SparkFun-Capacitors:CAP0603-CAP
- added C29: 5.6 pF, SparkFun-Capacitors:CAP0603-CAP
- added C30: 1 uF, SparkFun-Capacitors:CAP0603-CAP
- added C33: 33 nF, SparkFun-Capacitors:CAP0603-CAP
- added C38: 1.5 pF, SparkFun-Capacitors:CAP0603-CAP
- added C39: 2.2 nF, SparkFun-Capacitors:CAP0603-CAP
- added C40: 4.7 pF, SparkFun-Capacitors:CAP0603-CAP
- added C41: 1.0 pF, SparkFun-Capacitors:CAP0603-CAP
- added C42, C43: 22 pF, SparkFun-Capacitors:CAP0603-CAP
- added DS1, DS10, DS11, DS12, DS2, DS3, DS4, DS5, DS6, DS7, DS8, DS9: LTST-C19FD1WT, led:LTST-C19FD1WT
- added L3: 2.2uH, 1.4A, appfruits:LPS30152.2UH
- added L4, L5: DNP, SparkFun-Passives:INDUCTOR30OHM,1.8A
- added L6: 8.2 nH, SparkFun-Passives:INDUCTOR0402
- added L7: 3.9 nH, SparkFun-Passives:INDUCTOR0402
- added L8: 2.7 nH, SparkFun-Passives:INDUCTOR0402
- added LED3: (no value), appfruits:LED-GREEN
- added R10: 2M, appfruits:RESISTOR-2M
- added R11: 1.2M, appfruits:RESISTOR-1.2M
- added R12: 470, appfruits:RESISTOR-470
- added R13, R14: 220K, appfruits:RESISTOR-220K
- added R15, R16, R17, R18, R19, R20: 10k, SparkFun:RESISTOR0603-RES
- added R21, R22, R23, R24, R25, R26, R27, R28, R29, R30, R31, R32, R33, R34, R35, R36, R37, R38, R39, R40, R41, R42, R43, R44, R45, R46, R47, R48, R49, R50, R51, R52: (no value), SparkFun:RESISTOR0402-RES
- added R53, R54, R56: 12k, SparkFun-Resistors:RESISTOR0603-RES
- added R55: 200, SparkFun-Resistors:RESISTOR0603-RES
- added R57: 10k, SparkFun-Resistors:RESISTOR0603-RES
- added R58: 22k, SparkFun-Resistors:RESISTOR0603-RES
- added R59: 1M, SparkFun-Resistors:RESISTOR0603-RES
- added U2: TPS61200, appfruits:TPS61200
- added U3, U4: PCA9552BS, NXP_By_element14_Batch_1:PCA9552BS
- added U5: MPU-9250, chips:MPU-9250
- added U6: 25Q40, wifi:25Q40
- added U7: ESP8266EX, wifi:ESP8266EX
- added U8: NRF24L01, RF:NRF24L01
- added Y3: 26 Mhz, SparkFun-FreqCtrl:CRYSTAL5X3
- added Y4: 16 Mhz, SparkFun-FreqCtrl:CRYSTAL5X3
- C1, C7: value 2.2uF -> 0.1uF; device appfruits:CAPACITOR-2.2UF -> appfruits:CAPACITOR-0.1UF
- C5, C6: value 0.1uF -> 2.2uF; device appfruits:CAPACITOR-0.1UF -> appfruits:CAPACITOR-2.2UF
- R2, R3: value (none) -> 470; device SparkFun:RESISTOR0402-RES -> appfruits:RESISTOR-470
- R4, R5: value (none) -> 10k; device SparkFun:RESISTOR0402-RES -> SparkFun-Resistors:RESISTOR0603-RES
- R6, R7: value 470 -> (none); device appfruits:RESISTOR-470 -> SparkFun:RESISTOR0402-RES
- R8, R9: value 10k -> (none); device SparkFun-Resistors:RESISTOR0603-RES -> SparkFun:RESISTOR0402-RES
Connections:
- removed net VCC: C1.1, C2.1, C5.1, C7.1
- removed net V_OUT: C3.1, R7.2, R9.1
- new net !CS: U1.PTC2/ADC0_SE12, U5.!CS
- new net !RESET0: U1.PTA4, U3.!RESET
- new net !RESET1: U1.PTA5, U4.!RESET
- new net CLK: R55.1, U6.CLK
- new net CS: U6.CS#, U7.SD_CMD/20
- new net DIO: U6.DIO, U7.SD_DATA_1/23
- new net DO: U6.DO, U7.SD_DATA_0/22
- new net HOLD#: U6.HOLD#, U7.SD_DATA_2/18
- new net N$100: C26.1, U7.XTAL_IN/28, Y3.2
- new net N$101: AE1.SIGNAL, C29.1, L4.1
- new net N$102: R56.2, U7.MTCK/12
- new net N$103: R57.2, U7.MTDO/13
- new net N$107: R53.1, U7.RES12K/31
- new net N$108: C42.1, R59.1, U8.XC2/9, Y4.1
- new net N$109: C43.1, R59.2, U8.XC1/10, Y4.2
- new net N$111: L6.1, L7.1, U8.ANT2/13
- new net N$112: R58.1, U8.IREF/16
- new net N$113: C33.2, U8.DVDD/19
- new net N$114: L6.2, L8.1, U8.ANT1/12
- new net N$115: AE2.SIGNAL, C38.2, C41.1
- new net N$116: C38.1, L7.2
- new net N$117: C39.1, C40.1, L8.2, U8.VDD_PA/11
- new net N$118: C32.2, U7.VDD3P3/4, U7.VDD_RTC/5
- new net N$22: C29.2, L5.1, U7.LNA/2
- new net N$23: C27.1, U7.XTAL_OUT/27, Y3.1
- new net N$24: L3.1, U2.L
- new net N$25: C15.1, U2.VAUX
- new net N$26: C13.2, R10.1, R13.2, U2.UVLO
- new net N$27: R11.1, R14.2, U2.FB
- new net N$28: LED3.A, R12.2
- new net N$30: R16.1, U3.A1
- new net N$31: R17.1, U3.A0
- new net N$32: R18.1, U4.A2
- new net N$33: R19.1, U4.A1
- new net N$34: R20.1, U4.A0
- new net N$35: R15.1, U3.A2
- new net N$36: DS9.R, R44.2
- new net N$37: DS7.R, R39.2
- new net N$38: DS7.B, R40.2
- new net N$39: DS7.G, R37.2
- new net N$40: DS9.B, R46.2
- new net N$41: DS9.G, R42.2
- new net N$42: DS2.G, R25.2
- new net N$43: DS2.B, R22.2
- new net N$44: DS11.B, R51.2
- new net N$45: DS11.G, R48.2
- new net N$46: R21.1, U3.LED0
- new net N$47: DS3.R, R28.2
- new net N$48: R23.1, U3.LED1
- new net N$49: R24.1, U3.LED2
- new net N$50: DS10.B, R43.2
- new net N$51: DS1.R, R23.2
- new net N$52: DS4.R, R29.2
- new net N$53: DS1.B, R24.2
- new net N$54: DS1.G, R21.2
- new net N$55: DS3.B, R30.2
- new net N$56: DS3.G, R26.2
- new net N$57: DS12.G, R52.2
- new net N$58: DS6.B, R33.2
- new net N$59: DS8.G, R41.2
- new net N$60: R26.1, U3.LED3
- new net N$61: DS4.G, R31.2
- new net N$62: DS10.G, R47.2
- new net N$63: DS4.B, R27.2
- new net N$64: DS6.G, R36.2
- new net N$65: DS5.B, R35.2
- new net N$66: DS5.G, R32.2
- new net N$67: DS10.R, R45.2
- new net N$68: DS8.B, R38.2
- new net N$69: R28.1, U3.LED4
- new net N$70: DS12.B, R49.2
- new net N$71: R30.1, U3.LED5
- new net N$72: R32.1, U3.LED6
- new net N$73: R35.1, U3.LED7
- new net N$74: R37.1, U3.LED8
- new net N$75: R39.1, U3.LED9
- new net N$76: R40.1, U3.LED10
- new net N$77: R42.1, U3.LED11
- new net N$78: R44.1, U3.LED12
- new net N$79: R46.1, U3.LED13
- new net N$80: R48.1, U3.LED14
- new net N$81: R51.1, U3.LED15
- new net N$82: DS6.R, R34.2
- new net N$83: DS12.R, R50.2
- new net N$84: R22.1, U4.LED15
- new net N$85: R25.1, U4.LED14
- new net N$86: R27.1, U4.LED13
- new net N$87: R29.1, U4.LED12
- new net N$88: R31.1, U4.LED11
- new net N$89: R33.1, U4.LED10
- new net N$90: R34.1, U4.LED9
- new net N$91: R36.1, U4.LED8
- new net N$92: R38.1, U4.LED7
- new net N$93: R41.1, U4.LED6
- new net N$94: R43.1, U4.LED5
- new net N$95: R45.1, U4.LED4
- new net N$96: R47.1, U4.LED3
- new net N$97: R49.1, U4.LED2
- new net N$98: R50.1, U4.LED1
- new net N$99: R52.1, U4.LED0
- new net SCL: R4.2, U1.PTB2/I2C0_SCL, U3.SCL, U4.SCL, U5.SCLK
- new net WP#: U6.WP#, U7.SD_DATA_3/19
- net 3.3V: now also C1.1, C16.1, C17.1, C18.1, C19.1, C20.1, C21.2, C22.1, C24.1, C25.1, C28.2, C30.2, C31.2, C34.1, C35.1, C36.1, C37.1, DS1.V, DS10.V, DS11.V, DS12.V, DS2.V, DS3.V, DS4.V, DS5.V, DS6.V, DS7.V, DS8.V, DS9.V, R1.1, R11.2, R12.1, R20.2, R54.2, TP12.TP, TP15.TP, TP19.TP, TP25.TP, TP3.TP, TP31.TP, TP6.TP, TP9.TP, U2.VOUT, U3.VDD, U4.VDD, U5.VDD, U5.VDDIO, U6.VCC, U7.VDD3P3/3, U7.VDDA/1, U7.VDDA/30, U7.VDDD/29, U7.VDDPST/11, U7.VDDPST/17, U8.VDD/15, U8.VDD/18, U8.VDD/7; no longer C7.1, R9.1, TP17.TP, TP22.TP, TP23.TP, TP28.TP, TP29.TP, TP34.TP, TP35.TP, TP4.TP
- net CE: now also U1.PTC9/ADC1_SE5B, U8.CE/1; no longer U1.PTC9
- net CHIP_EN: now also U1.PTC1/ADC0_SE15, U7.CHIP_EN/7; no longer U1.PTC1
- net CSN: now also U1.PTC4/SPI0_PCS0, U8.CSN/2; no longer U1.PTC4
- net FSYNC: now also U1.PTB1/ADC0_SE9, U5.FSYNC; no longer U1.PTB1
- net GND: now also C14.2, C15.2, C16.2, C17.2, C18.2, C19.2, C20.2, C21.1, C22.2, C23.1, C24.2, C25.2, C26.2, C27.2, C28.1, C30.1, C31.1, C32.1, C33.1, C34.2, C35.2, C36.2, C37.2, C39.2, C40.2, C41.2, C42.2, C43.2, L4.2, L5.2, LED3.C, R13.1, R14.1, R15.2, R16.2, R17.2, R18.2, R19.2, R53.2, R56.1, R57.1, R58.2, R9.1, TP11.TP, TP14.TP, TP17.TP, TP23.TP, TP29.TP, TP35.TP, TP5.TP, TP8.TP, U2.GND, U2.PAD@1, U2.PAD@2, U2.PAD@3, U2.PAD@4, U2.PAD@5, U2.PGND, U3.VSS, U4.VSS, U5.AD0/MISO, U5.GND, U6.GND, U7.GND, U8.VSS/14, U8.VSS/17, U8.VSS/20, U8.VSS/8; no longer C10.2, C12.2, C7.2, C8.1, C9.2, LED1.C, R1.2, R3.1, R4.1, R5.1, R6.1, TP1.TP, TP19.TP, TP21.TP, TP25.TP, TP27.TP, TP3.TP, TP31.TP, TP33.TP
- net GPIO0: now also U1.PTB18/CAN0_RX, U7.GPIO0/15; no longer U1.PTB18
- net GPIO2: now also U1.PTB19/CAN0_TX, U7.GPIO2/14; no longer U1.PTB19
- net INT: now also U1.PTB0/ADC0_SE8, U5.INT; no longer U1.PTB0
- net IRQ: now also U1.PTC8/ADC1_SE4B, U8.IRQ/6; no longer U1.PTC8
- net MISO: now also U1.PTC7/SPI0_SIN, U8.MISO/5; no longer U1.PTC7
- net MOSI: now also U1.PTC6/SPI0_SOUT, U8.MOSI/4; no longer U1.PTC6
- net N$1: no longer C10.1, C9.1, L1.1, L2.2
- net N$10: now also U1.PTD6/UART0_RX; no longer U1.PTD6
- net N$11: now also TP33.TP; no longer C7.1, TP9.TP
- net N$12: now also TP22.TP; no longer C8.2, TP5.TP
- net N$13: now also U1.PTD7/UART0_TX; no longer L2.1, U1.PTD7
- net N$14: now also TP28.TP; no longer C12.1, C6.1, TP6.TP
- net N$15: now also TP34.TP; no longer TP10.TP
- net N$16: now also TP16.TP; no longer R5.2, TP11.TP
- net N$17: now also TP7.TP; no longer TP12.TP
- net N$18: now also TP10.TP; no longer TP13.TP
- net N$19: now also TP13.TP; no longer TP14.TP
- net N$2: no longer C4.1
- net N$20: now also TP4.TP; no longer TP15.TP
- net N$21: now also TP1.TP; no longer TP16.TP
- net N$29: now also R2.2; no longer R7.2
- net N$3: now also R55.2, U7.SD_CLK/21; no longer C2.2, R3.1, R4.2, U1.PTC2
- net N$4: now also C23.2, U5.REGOUT; no longer R6.2, R7.1, R8.2, U1.PTB2
- net N$5: now also TP21.TP; no longer LED1.A, R9.2, TP7.TP
- net N$6: now also TP27.TP; no longer TP8.TP
- net N$7: now also R1.2; no longer C6.2, R6.2
- net N$8: no longer R1.1
- net PTA0: now also R9.2; no longer R3.2
- net PTA1: now also R7.2; no longer R4.2
- net PTA3: now also R6.2; no longer R2.2
- net RESET_B: now also R8.2; no longer R5.2
- net SCK: now also U1.PTC5/SPI0_SCK, U8.SCK/3; no longer U1.PTC5
- net SDA: now also R5.2, U1.PTB3/I2C0_SDA, U3.SDA, U4.SDA, U5.SDA/MOSI; no longer R9.2, U1.PTB3
- net U0RX: now also U1.PTB17/UART0_TX, U7.U0RXD/25; no longer U1.PTB17
- net U0TX: now also U1.PTB16/UART0_RX, U7.U0TXD/26; no longer U1.PTB16
- net VDDA: now also C6.1, R3.1; no longer C1.1, R1.1
- net VREFH: now also C7.1, R3.2; no longer C6.1, R1.2
- net VREFL: now also C7.2; no longer C1.2
- net V_IN: now also C13.1, C14.1, L3.2, R10.2, U2.EN, U2.PS, U2.VIN; no longer C1.1, C2.1, L1.2, R3.2
- net WIFI_RESET: now also R54.1, U1.PTC0/ADC0_SE14, U7.EXT_RSTB/32; no longer U1.PTC0
- net XPD_DCDC: now also U1.PTC3/CMP1_IN1, U7.XPD_DCDC/8; no longer U1.PTC3
Other:
- note added: "+Z Accelerometer -Z Compass"
- note added: "0: X- Group"
- note added: "1: X+ Group"
- note added: "2: Y- Group"
- note added: "3: Y+ Group"
- note added: "Group 0"
- note added: "Group 1"
- note added: "Group 2"
- note added: "Group 3"
- note added: "I/O Groups: Place at board edge as noted by group name. Place the I/O towards the inside. Place ground at the board edge. Place power in between. See LED_DRIVER block for LEDS to be placed near these ports."
- note added: "Inductor minimum value: Vin_max * .5(us/A) 4.2v * .5 (us/A) = 2.1uH Max Inductor Current = 743mA"
- note added: "Input dropout voltage of ~2.5v R_uv3 = R_uv4 * (Vin_min / V_uvlo - 1) 2M = 220k * (2.5V / .25v - 1)"
- note added: "NOTES"
- note added: "Output of 3.3v R_fb1 = R_fb2 x (Vout/Vfb - 1) 1.2M = 220k * (3.3v/.5v - 1)"
- note added: "Place decoupling caps near VDD pins."
- note added: "Power inlet: Single cell Li-Po battery, or any power source where 2.5 < Vout < 7v See sheet 2 for regulator circuit."
- note added: "R_fb1"
- note added: "R_fb2"
- note added: "R_uv3"
- note added: "R_uv4"
- note added: "Refer to sheet 1 for GPIO blocks. Place three LEDs as grouped next to each GPIO block."
- note added: "Source"
- note removed: "FIX THIS PINOUT"
- note removed: "I/O Groups: Place at board edge as noted by group name. Place the I/O towards the inside. Place ground at the board edge. Place power in between."
- note removed: "Switch for VIN from LiPO to VCC into regulator"
- note removed: "UVLO 2.6V"
- note removed: "X+ Group"
- note removed: "X- Group"
- note removed: "Y+ Group"
- note removed: "Y- Group"

Commit message: Mas cleanup
Other:
- note added: "I/O Groups: Place at board edge as noted by group name. Place the I/O towards the inside. Place ground at the board edge. Place power in between. See LED drivers on page 3 for LED groups to be placed near these ports."
- note removed: "I/O Groups: Place at board edge as noted by group name. Place the I/O towards the inside. Place ground at the board edge. Place power in between. See LED_DRIVER block for LEDS to be placed near these ports."
Changed lines of the file:
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@@
 <setting verticaltext="up"/>
 </settings>
-<grid distance="0.1" unitdist="inch" unit="inch" style="dots" multiple="1" display="no" altdistance="0.01" altunitdist="inch" altunit="inch"/>
+<grid distance="0.05" unitdist="inch" unit="inch" style="dots" multiple="1" display="yes" altdistance="0.01" altunitdist="inch" altunit="inch"/>
 <layers>
 <layer number="1" name="Top" color="4" fill="1" visible="no" active="no"/>
@@
 Place ground at the board edge.
 Place power in between.
-See LED_DRIVER block for LEDS to be placed
-near these ports.</text>
+See LED drivers on page 3 for LED groups to be
+placed near these ports.</text>
 <wire x1="259.08" y1="-191.77" x2="205.74" y2="-191.77" width="0.1524" layer="97"/>
 <wire x1="205.74" y1="-191.77" x2="205.74" y2="-248.92" width="0.1524" layer="97"/>
@@
 <segment>
 <pinref part="U1" gate="G$1" pin="PTA5"/>
-<wire x1="201.93" y1="-179.07" x2="262.89" y2="-179.07" width="0.1524" layer="91"/>
-<label x="262.89" y="-179.07" size="1.778" layer="95" xref="yes"/>
+<wire x1="201.93" y1="-179.07" x2="246.38" y2="-179.07" width="0.1524" layer="91"/>
+<wire x1="246.38" y1="-179.07" x2="246.38" y2="-180.34" width="0.1524" layer="91"/>
+<wire x1="246.38" y1="-180.34" x2="262.89" y2="-180.34" width="0.1524" layer="91"/>
+<label x="262.89" y="-180.34" size="1.778" layer="95" xref="yes"/>
 </segment>
 </net>
@@
 <wire x1="201.93" y1="-163.83" x2="246.38" y2="-163.83" width="0.1524" layer="91"/>
 <pinref part="R5" gate="G$1" pin="2"/>
-<wire x1="246.38" y1="-163.83" x2="262.89" y2="-163.83" width="0.1524" layer="91"/>
+<wire x1="246.38" y1="-163.83" x2="246.38" y2="-165.1" width="0.1524" layer="91"/>
+<wire x1="246.38" y1="-165.1" x2="262.89" y2="-165.1" width="0.1524" layer="91"/>
 <wire x1="246.38" y1="-160.02" x2="246.38" y2="-163.83" width="0.1524" layer="91"/>
 <junction x="246.38" y="-163.83"/>
-<label x="262.89" y="-163.83" size="1.778" layer="95" xref="yes"/>
-</segment>
-</net>
+<label x="262.89" y="-165.1" size="1.778" layer="95" xref="yes"/>
+</segment>
+</net>
