File: Circuit/P1R5/P1R5.sch (EAGLE design)
At the start: 178 parts, among them J1 2X5_0.05"_CORTEX_DEBUGTH_NOKE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, U1 MK20DX256VLH7, U2 TPS61200, U3 PCA9552BS, U4 PCA9552BS, U5 MPU-9250, U6 25Q40, U7 ESP8266EX, U8 NRF24L01, Y1 16Mhz/8pF, Y2 32.768KHz, Y3 26 Mhz, Y4 16 Mhz

Commit message: Matched all parts to bom-ex db.
Parts:
- removed LED1, LED2, LED3: (no value), appfruits:LED-GREEN
- added DS13, DS14, DS15: LTST-C19FD1WT, led:LTST-C19FD1WT
- added TP37, TP38, TP39, TP40, TP41, TP42, TP43, TP44, TP45, TP46, TP47, TP48, TP49, TP50, TP51, TP52, TP53, TP54, TP55, TP56, TP57, TP58: TPPAD1-20, testpad:TPPAD1-20
- AE1, AE2: value ANTENNA2SMD -> 2450AT18A100E; PARTNO (none) -> 2450AT18A100E
- C1, C15, C2, C3, C36, C4, C7, C8: device appfruits:CAPACITOR-0.1UF -> SparkFun-Capacitors:CAP0402-CAP; PARTNO (none) -> C1005X7R1C104K050BC
- C10: device appfruits:CAPACITOR-10UF -> SparkFun-Capacitors:CAP0603-CAP; PARTNO (none) -> C1608X7S0J106M080AC
- C11, C14, C9: value 10uF -> 0.1uF; device appfruits:CAPACITOR-10UF -> SparkFun-Capacitors:CAP0402-CAP; PARTNO (none) -> C1005X7R1C104K050BC
- C12: value 10uF -> 22uF; device appfruits:CAPACITOR-10UF -> SparkFun-Capacitors:CAP1210; PARTNO (none) -> C3225X7R1A226K230AC
- C13: value 0.1uF -> 22uF; device appfruits:CAPACITOR-0.1UF -> SparkFun-Capacitors:CAP1210; PARTNO (none) -> C3225X7R1A226K230AC
- C16: value 22uF -> 10uF; device appfruits:CAPACITOR-22UF -> SparkFun-Capacitors:CAP0603-CAP; PARTNO (none) -> C1608X7S0J106M080AC
- C17: value 0.1uF -> 10uF; device appfruits:CAPACITOR-0.1UF -> SparkFun-Capacitors:CAP0603-CAP; PARTNO (none) -> C1608X7S0J106M080AC
- C18, C20: value 2.2uF -> 0.1 uF; device appfruits:CAPACITOR-2.2UF -> SparkFun-Capacitors:CAP0402-CAP; PARTNO (none) -> C1005X7R1C104K050BC
- C19: value 0.1uF -> 0.1 uF; device appfruits:CAPACITOR-0.1UF -> SparkFun-Capacitors:CAP0402-CAP; PARTNO (none) -> C1005X7R1C104K050BC
- C21, C25, C32: value .1 uF -> 10uF; PARTNO (none) -> C1608X7S0J106M080AC
- C22, C23, C31, C34, C35: value .1 uF -> 0.1 uF; device SparkFun-Capacitors:CAP0603-CAP -> SparkFun-Capacitors:CAP0402-CAP; PARTNO (none) -> C1005X7R1C104K050BC
- C24: value .1 uF -> 15 pF; device SparkFun-Capacitors:CAP0603-CAP -> SparkFun-Capacitors:CAP0402-CAP; PARTNO (none) -> C1005C0G1H150J050BA
- C26: device SparkFun-Capacitors:CAP0603-CAP -> SparkFun-Capacitors:CAP0402-CAP; PARTNO (none) -> C1005C0G1H150J050BA
- C27: value 15 pF -> 0.1 uF; device SparkFun-Capacitors:CAP0603-CAP -> SparkFun-Capacitors:CAP0402-CAP; PARTNO (none) -> C1005X7R1C104K050BC
- C28: value .1 uF -> 5.6 pF; device SparkFun-Capacitors:CAP0603-CAP -> SparkFun-Capacitors:CAP0402-CAP; PARTNO (none) -> GRM1555C1H5R6CA01D
- C29: value 5.6 pF -> 0.1 uF; device SparkFun-Capacitors:CAP0603-CAP -> SparkFun-Capacitors:CAP0402-CAP; PARTNO (none) -> C1005X7R1C104K050BC
- C30: value 1 uF -> 0.1 uF; device SparkFun-Capacitors:CAP0603-CAP -> SparkFun-Capacitors:CAP0402-CAP; PARTNO (none) -> C1005X7R1C104K050BC
- C33: value 33 nF -> .033 uF; device SparkFun-Capacitors:CAP0603-CAP -> SparkFun-Capacitors:CAP0402-CAP; PARTNO (none) -> C1005X7R1H333K050BB
- C37, C5, C6: value 2.2uF -> 10uF; device appfruits:CAPACITOR-2.2UF -> SparkFun-Capacitors:CAP0603-CAP; PARTNO (none) -> C1608X7S0J106M080AC
- C38: device SparkFun-Capacitors:CAP0603-CAP -> SparkFun-Capacitors:CAP0402-CAP; PARTNO (none) -> C1005C0G1H1R5B050BA
- C39: value 2.2 nF -> 2200 pF; device SparkFun-Capacitors:CAP0603-CAP -> SparkFun-Capacitors:CAP0402-CAP; PARTNO (none) -> C1005X7R1H222K050BA
- C40: device SparkFun-Capacitors:CAP0603-CAP -> SparkFun-Capacitors:CAP0402-CAP; PARTNO (none) -> CGA2B2C0G1H4R7C050BA
- C41: device SparkFun-Capacitors:CAP0603-CAP -> SparkFun-Capacitors:CAP0402-CAP; PARTNO (none) -> C1005C0G1H010B050BA
- C42, C43: device SparkFun-Capacitors:CAP0603-CAP -> SparkFun-Capacitors:CAP0402-CAP; PARTNO (none) -> C1005C0G1H220J050BA
- DS1, DS2, DS3: value LTST-C19FD1WT -> LTST-C191TBKT; device led:LTST-C19FD1WT -> appfruits:LED-GREEN; PARTNO (none) -> LTST-C191TBKT
- DS10, DS11, DS12, DS4, DS5, DS6, DS7, DS8, DS9: PARTNO (none) -> LTST-C19FD1WT
- J1: PARTNO (none) -> 20021111-00010T4LF
- JP1: value (none) -> M20PTH; PARTNO (none) -> M20PTH
- L1, L2: PARTNO (none) -> BK2125HM601-T
- L3: PARTNO (none) -> LPS3015-222MRB
- L4, L5, L6, L7, L8: PARTNO (none) -> DNP
- R1, R12, R2, R3: device appfruits:RESISTOR-470 -> appfruits:RESISTOR0402; PARTNO (none) -> ERJ-3GEYJ471V
- R10: device appfruits:RESISTOR-2M -> appfruits:RESISTOR0402; PARTNO (none) -> ERJ-3GEYJ205V
- R11: device appfruits:RESISTOR-1.2M -> appfruits:RESISTOR0402; PARTNO (none) -> ERJ-3GEYJ125V
- R13, R14: device appfruits:RESISTOR-220K -> appfruits:RESISTOR0402; PARTNO (none) -> ERJ-3GEYJ224V
- R15, R16, R17, R18, R19, R20: device SparkFun:RESISTOR0603-RES -> appfruits:RESISTOR0402; PARTNO (none) -> *
- R21, R22, R23, R24, R25, R26, R27, R28, R29, R30, R31, R32, R33, R34, R35, R36, R37, R38, R39, R40, R41, R42, R43, R44, R45, R46, R47, R48, R49, R50, R51, R52: value (none) -> 86.6; device SparkFun:RESISTOR0402-RES -> appfruits:RESISTOR0402; PARTNO (none) -> 5-1879213-0
- R4, R5, R53, R54, R55, R56, R57, R58, R59: device SparkFun-Resistors:RESISTOR0603-RES -> appfruits:RESISTOR0402; PARTNO (none) -> *
- R6, R7, R8, R9: value (none) -> 10k; device SparkFun:RESISTOR0402-RES -> appfruits:RESISTOR0402; PARTNO (none) -> *
- S1: value (none) -> CUS-12TB; PARTNO (none) -> CUS-12TB
- TP1, TP10, TP11, TP12, TP13, TP14, TP15, TP16, TP17, TP18, TP19, TP2, TP20, TP21, TP22, TP23, TP24, TP25, TP26, TP27, TP28, TP29, TP3, TP30, TP31, TP32, TP33, TP34, TP35, TP36, TP4, TP5, TP6, TP7, TP8, TP9: PARTNO (none) -> TEST POINT
- U1: PARTNO (none) -> MK20DX256VLH7
- U2: PARTNO (none) -> TPS61200DRCR
- U3, U4: PARTNO (none) -> PCA9552BS
- U5: PARTNO (none) -> MPU-9250
- U6: PARTNO (none) -> 25Q40
- U7: PARTNO (none) -> ESP8266EX
- U8: PARTNO (none) -> NRF24L01P-T
- Y1: value 16Mhz/8pF -> 8MHz; device appfruits:CRYSTAL/SMD-5X3-GND16MHZ/8PF -> CrystalOscillators:ASCO.063X.047; MF ECS -> (none); MPN ECS-160-8-30B-CKM -> (none); PARTNO (none) -> ASCO-8.000MHZ-EK-T3
- Y2: value 32.768KHz -> 34.728kHz; device appfruits:CRYSTAL/32.768KHZ/SMD-TXC_7A -> CrystalOscillators:ABS06ABS06_.079X.047; MF Epson Timing -> (none); MPN FC-255 32.7680K-A3 -> (none); PARTNO (none) -> ABS06-32.768KHZ-T
- Y3, Y4: PARTNO (none) -> *
Connections:
- net !CS: now also TP44.TP
- net !RESET0: now also TP39.TP
- net !RESET1: now also TP40.TP
- net 3.3V: now also C12.1, C13.1, C14.1, C15.1, C18.2, C21.1, C23.1, C27.2, C29.2, C32.1, DS13.V, DS14.V, DS15.V, Y1.VCC; no longer C18.1, C20.1, C21.2, C24.1, C28.2, C31.2, DS1.V, DS2.V, DS3.V
- net CE: now also TP58.TP
- net CHIP_EN: now also TP50.TP
- net CSN: now also TP57.TP
- net FSYNC: now also TP41.TP
- net GND: now also C10.2, C11.2, C12.2, C13.2, C18.1, C20.1, C21.2, C23.2, C27.1, C29.1, C32.2, DS3.C, Y1.GND; no longer C10.1, C11.1, C12.1, C18.2, C20.2, C21.1, C23.1, C27.2, C28.1, C32.1, C9.1, LED3.C
- net GPIO0: now also TP52.TP
- net GPIO2: now also TP51.TP
- net INT: now also TP45.TP
- net IRQ: now also TP53.TP
- net MISO: now also TP54.TP
- net MOSI: now also TP55.TP
- net N$1: now also U1.PTA18/EXTAL0, Y1.OUT; no longer C11.2, U1.XTAL32, Y2.2
- net N$10: now also DS1.C; no longer LED1.C
- net N$100: now also C24.1; no longer C26.1
- net N$101: now also C28.1; no longer C29.1
- net N$118: now also C31.2; no longer C32.2
- net N$13: now also DS2.C; no longer LED2.C
- net N$2: now also U1.PTA19/XTAL0, Y1.ENABLE; no longer C12.2, U1.EXTAL32, Y2.1
- net N$22: now also C28.2; no longer C29.2
- net N$23: now also C26.1; no longer C27.1
- net N$25: now also C11.1; no longer C15.1
- net N$26: now also C9.2; no longer C13.2
- net N$28: now also DS3.A; no longer LED3.A
- net N$29: now also DS2.A; no longer LED2.A
- net N$36: now also DS12.R; no longer DS9.R
- net N$37: now also DS10.R; no longer DS7.R
- net N$38: now also DS10.B; no longer DS7.B
- net N$39: now also DS10.G; no longer DS7.G
- net N$4: now also C20.2; no longer C23.2
- net N$40: now also DS12.B; no longer DS9.B
- net N$41: now also DS12.G; no longer DS9.G
- net N$42: now also DS5.G; no longer DS2.G
- net N$43: now also DS5.B; no longer DS2.B
- net N$44: now also DS14.B; no longer DS11.B
- net N$45: now also DS14.G; no longer DS11.G
- net N$47: now also DS6.R; no longer DS3.R
- net N$50: now also DS13.B; no longer DS10.B
- net N$51: now also DS4.R; no longer DS1.R
- net N$52: now also DS7.R; no longer DS4.R
- net N$53: now also DS4.B; no longer DS1.B
- net N$54: now also DS4.G; no longer DS1.G
- net N$55: now also DS6.B; no longer DS3.B
- net N$56: now also DS6.G; no longer DS3.G
- net N$57: now also DS15.G; no longer DS12.G
- net N$58: now also DS9.B; no longer DS6.B
- net N$59: now also DS11.G; no longer DS8.G
- net N$61: now also DS7.G; no longer DS4.G
- net N$62: now also DS13.G; no longer DS10.G
- net N$63: now also DS7.B; no longer DS4.B
- net N$64: now also DS9.G; no longer DS6.G
- net N$65: now also DS8.B; no longer DS5.B
- net N$66: now also DS8.G; no longer DS5.G
- net N$67: now also DS13.R; no longer DS10.R
- net N$68: now also DS11.B; no longer DS8.B
- net N$7: now also DS1.A; no longer LED1.A
- net N$70: now also DS15.B; no longer DS12.B
- net N$8: now also U1.XTAL32, Y2.2; no longer C9.2, U1.PTA18/EXTAL0, Y1G$1.2
- net N$82: now also DS9.R; no longer DS6.R
- net N$83: now also DS15.R; no longer DS12.R
- net N$9: now also U1.EXTAL32, Y2.1; no longer C10.2, U1.PTA19/XTAL0, Y1G$1.1
- net SCK: now also TP56.TP
- net SCL: now also R5.2, TP42.TP; no longer R4.2
- net SDA: now also R4.2, TP37.TP, TP38.TP, TP43.TP; no longer R5.2
- net U0RX: now also TP47.TP
- net U0TX: now also TP46.TP
- net V_IN: now also C10.1, C9.1; no longer C13.1, C14.1
- net WIFI_RESET: now also TP48.TP
- net XPD_DCDC: now also TP49.TP
Other:
- note added: "To IMU, page 4"
- note added: "To LEDs on page 3 and IMU on page 4"
- note added: "To LEDs, page 3"
- note added: "To Mesh, page 6"
- note added: "To WiFi, page 5"
