File: Circuit/P1R5/P1R5.sch (EAGLE design)
At the start: 200 parts, among them J1 2X5_0.05"_CORTEX_DEBUGTH_NOKE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, U1 MK20DX256VLH7, U2 TPS61200, U3 PCA9552BS, U4 PCA9552BS, U5 MPU-9250, U6 25Q40, U7 ESP8266EX, U8 NRF24L01, Y1 8MHz, Y2 34.728kHz, Y3 26 Mhz, Y4 16 Mhz

Commit message: Began laying out PCB
Parts:
- removed C42, C43: 22 pF, SparkFun-Capacitors:CAP0402-CAP
- C10: value 10uF -> 22uF; device SparkFun-Capacitors:CAP0603-CAP -> SparkFun-Capacitors:CAP1210; PARTNO C1608X7S0J106M080AC -> C3225X7R1A226K230AC
- C11: value 0.1uF -> 22uF; device SparkFun-Capacitors:CAP0402-CAP -> SparkFun-Capacitors:CAP1210; PARTNO C1005X7R1C104K050BC -> C3225X7R1A226K230AC
- C12, C13: value 22uF -> 0.1uF; device SparkFun-Capacitors:CAP1210 -> SparkFun-Capacitors:CAP0402-CAP; PARTNO C3225X7R1A226K230AC -> C1005X7R1C104K050BC
- C14, C15, C4, C8: value 0.1uF -> 10uF; device SparkFun-Capacitors:CAP0402-CAP -> SparkFun-Capacitors:CAP0603-CAP; PARTNO C1005X7R1C104K050BC -> C1608X7S0J106M080AC
- C16, C17, C21, C25, C32: value 10uF -> 0.1 uF; device SparkFun-Capacitors:CAP0603-CAP -> SparkFun-Capacitors:CAP0402-CAP; PARTNO C1608X7S0J106M080AC -> C1005X7R1C104K050BC
- C19, C23, C30, C35: value 0.1 uF -> 10uF; device SparkFun-Capacitors:CAP0402-CAP -> SparkFun-Capacitors:CAP0603-CAP; PARTNO C1005X7R1C104K050BC -> C1608X7S0J106M080AC
- C22: value 0.1 uF -> 15 pF; PARTNO C1005X7R1C104K050BC -> C1005C0G1H150J050BA
- C26: value 15 pF -> 5.6 pF; PARTNO C1005C0G1H150J050BA -> GRM1555C1H5R6CA01D
- C28: value 5.6 pF -> 0.1 uF; PARTNO GRM1555C1H5R6CA01D -> C1005X7R1C104K050BC
- C31: value 0.1 uF -> .033 uF; PARTNO C1005X7R1C104K050BC -> C1005X7R1H333K050BB
- C33: value .033 uF -> 0.1 uF; PARTNO C1005X7R1H333K050BB -> C1005X7R1C104K050BC
- C34: value 0.1 uF -> 0.1uF
- C36: value 0.1uF -> 1.5 pF; PARTNO C1005X7R1C104K050BC -> C1005C0G1H1R5B050BA
- C37: value 10uF -> 2200 pF; device SparkFun-Capacitors:CAP0603-CAP -> SparkFun-Capacitors:CAP0402-CAP; PARTNO C1608X7S0J106M080AC -> C1005X7R1H222K050BA
- C38: value 1.5 pF -> 4.7 pF; PARTNO C1005C0G1H1R5B050BA -> CGA2B2C0G1H4R7C050BA
- C39: value 2200 pF -> 1.0 pF; PARTNO C1005X7R1H222K050BA -> C1005C0G1H010B050BA
- C40: value 4.7 pF -> 22 pF; PARTNO CGA2B2C0G1H4R7C050BA -> C1005C0G1H220J050BA
- C41: value 1.0 pF -> 22 pF; PARTNO C1005C0G1H010B050BA -> C1005C0G1H220J050BA
- C6: value 10uF -> 0.1uF; device SparkFun-Capacitors:CAP0603-CAP -> SparkFun-Capacitors:CAP0402-CAP; PARTNO C1608X7S0J106M080AC -> C1005X7R1C104K050BC
- L3: PARTNO LPS3015-222MRB -> BRL3225T2R2M
- L6: PARTNO DNP -> L-07C8N2JV6T
- L7: PARTNO DNP -> L-07C3N9SV6T
- L8: PARTNO DNP -> L-07C2N7SV6T
- R1, R12, R2: value 470 -> 25; PARTNO ERJ-3GEYJ471V -> CRCW040224R9FKED
- R10: PARTNO ERJ-3GEYJ205V -> CRCW04022M00FKED
- R11: value 1.2M -> 220K; PARTNO ERJ-3GEYJ125V -> CRCW0402220KFKED
- R13: value 220K -> 1.2M; PARTNO ERJ-3GEYJ224V -> CRCW04021M20FKED
- R14: PARTNO ERJ-3GEYJ224V -> CRCW0402220KFKED
- R15, R16, R17, R18, R19, R20, R4, R5, R57, R6, R7, R8, R9: PARTNO * -> CRCW040210K0FKED
- R3: PARTNO ERJ-3GEYJ471V -> CRCW0402470RFKED
- R53, R54, R56: PARTNO * -> CRCW040212K0FKED
- R55: PARTNO * -> CRCW0402200RFKED
- R58: PARTNO * -> CRCW040222K0FKED
- R59: PARTNO * -> CRCW04021M00FKED
- Y3: PARTNO * -> 7M-26.000MAAJ-T
- Y4: PARTNO * -> 7B-16.000MAAJ-T
Connections:
- removed net N$110: JP1.1, S1.S
- new net N$104: JP1.1, S1.P
- net 3.3V: now also C10.1, C11.1, C16.2, C20.1, C25.2, C28.2, C30.1, C33.1, R13.2; no longer C16.1, C18.2, C22.1, C25.1, C29.2, C30.2, C36.1, C37.1, C5.1, R11.2
- net GND: now also C16.1, C20.2, C25.1, C28.1, C30.2, C33.2, C38.2, C8.2, C9.2, R11.1; no longer C16.2, C20.1, C25.2, C26.2, C30.1, C33.1, C36.2, C42.2, C43.2, C5.2, R13.1
- net N$100: now also C22.1; no longer C24.1
- net N$101: now also C26.1; no longer C28.1
- net N$108: now also C40.1; no longer C42.1
- net N$109: now also C41.1; no longer C43.1
- net N$113: now also C31.2; no longer C33.2
- net N$115: now also C36.2, C39.1; no longer C38.2, C41.1
- net N$116: now also C36.1; no longer C38.1
- net N$117: now also C37.1, C38.1; no longer C39.1, C40.1
- net N$118: now also C29.2; no longer C31.2
- net N$16: now also U1.PTC11/ADC1_SE7B; no longer U1.PTC11/I2C1_SDA
- net N$17: now also U1.PTC10/ADC1_SE6B; no longer U1.PTC10/I2C1_SCL
- net N$22: now also C26.2; no longer C28.2
- net N$23: now also C24.1; no longer C26.1
- net N$25: now also C9.1; no longer C11.1
- net N$26: now also R11.2; no longer C9.2, R13.2
- net N$27: now also R13.1; no longer R11.1
- net N$4: now also C18.2; no longer C20.2
- net VDDA: now also C5.1; no longer C6.1
- net VREFH: now also C6.1; no longer C7.1
- net VREFL: now also C5.2; no longer C8.2
- net VREF_OUT: now also C7.1; no longer C8.1
- net V_IN: now also C8.1, S1.S; no longer C10.1, C9.1, S1.P
Other:
- moved on the sheet: C1, C10, C11, C14, C15, C18, C2, C21, C22, C23, C24, C25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

Commit message: Got majority of PCB layout done.
Parts:
- removed C38: 4.7 pF, SparkFun-Capacitors:CAP0402-CAP
- removed C39: 1.0 pF, SparkFun-Capacitors:CAP0402-CAP
- removed C40, C41: 22 pF, SparkFun-Capacitors:CAP0402-CAP
- removed TP57, TP58: TPPAD1-20, testpad:TPPAD1-20
- C1, C6: value 0.1uF -> 10uF; device SparkFun-Capacitors:CAP0402-CAP -> SparkFun-Capacitors:CAP0603-CAP; PARTNO C1005X7R1C104K050BC -> C1608X7S0J106M080AC
- C19: value 10uF -> 5.6 pF; device SparkFun-Capacitors:CAP0603-CAP -> SparkFun-Capacitors:CAP0402-CAP; PARTNO C1608X7S0J106M080AC -> GRM1555C1H5R6CA01D
- C20, C27: value 0.1 uF -> 10uF; device SparkFun-Capacitors:CAP0402-CAP -> SparkFun-Capacitors:CAP0603-CAP; PARTNO C1005X7R1C104K050BC -> C1608X7S0J106M080AC
- C22: value 15 pF -> 0.1 uF; PARTNO C1005C0G1H150J050BA -> C1005X7R1C104K050BC
- C25: value 0.1 uF -> 15 pF; PARTNO C1005X7R1C104K050BC -> C1005C0G1H150J050BA
- C26: value 5.6 pF -> 0.1 uF; PARTNO GRM1555C1H5R6CA01D -> C1005X7R1C104K050BC
- C32, C33: value 0.1 uF -> 22 pF; PARTNO C1005X7R1C104K050BC -> C1005C0G1H220J050BA
- C34: value 0.1uF -> 2200 pF; PARTNO C1005X7R1C104K050BC -> C1005X7R1H222K050BA
- C35: value 10uF -> 4.7 pF; device SparkFun-Capacitors:CAP0603-CAP -> SparkFun-Capacitors:CAP0402-CAP; PARTNO C1608X7S0J106M080AC -> CGA2B2C0G1H4R7C050BA
- C37: value 2200 pF -> 1.0 pF; PARTNO C1005X7R1H222K050BA -> C1005C0G1H010B050BA
- C4, C5: value 10uF -> 0.1uF; device SparkFun-Capacitors:CAP0603-CAP -> SparkFun-Capacitors:CAP0402-CAP; PARTNO C1608X7S0J106M080AC -> C1005X7R1C104K050BC
- L7: value 3.9 nH -> 2.7 nH; PARTNO L-07C3N9SV6T -> L-07C2N7SV6T
- L8: value 2.7 nH -> 3.9 nH; PARTNO L-07C2N7SV6T -> L-07C3N9SV6T
- R1: value 25 -> 470; PARTNO CRCW040224R9FKED -> CRCW0402470RFKED
- R12: value 25 -> 1.2M; PARTNO CRCW040224R9FKED -> CRCW04021M20FKED
- R13: value 1.2M -> 220K; PARTNO CRCW04021M20FKED -> CRCW0402220KFKED
- R14: value 220K -> 25; PARTNO CRCW0402220KFKED -> CRCW040224R9FKED
- R15, R16, R17, R18, R19, R20: value 10k -> 86.6; PARTNO CRCW040210K0FKED -> 5-1879213-0
- R2: value 25 -> 10k; PARTNO CRCW040224R9FKED -> CRCW040210K0FKED
- R3: value 470 -> 10k; PARTNO CRCW0402470RFKED -> CRCW040210K0FKED
- R31, R32, R33, R34, R35, R36: value 86.6 -> 10k; PARTNO 5-1879213-0 -> CRCW040210K0FKED
- R55: value 200 -> 12k; PARTNO CRCW0402200RFKED -> CRCW040212K0FKED
- R56: value 12k -> 10k; PARTNO CRCW040212K0FKED -> CRCW040210K0FKED
- R57: value 10k -> 200; PARTNO CRCW040210K0FKED -> CRCW0402200RFKED
- R58: value 22k -> 1M; PARTNO CRCW040222K0FKED -> CRCW04021M00FKED
- R59: value 1M -> 22k; PARTNO CRCW04021M00FKED -> CRCW040222K0FKED
- R6, R7: value 10k -> 25; PARTNO CRCW040210K0FKED -> CRCW040224R9FKED
- TP1, TP10, TP11, TP12, TP13, TP14, TP15, TP16, TP17, TP18, TP19, TP2, TP20, TP21, TP22, TP23, TP24, TP25, TP26, TP27, TP28, TP29, TP3, TP30, TP31, TP32, TP33, TP34, TP35, TP36, TP37, TP38, TP39, TP4, TP40, TP41, TP42, TP43, TP44, TP45, TP46, TP47, TP48, TP49, TP5, TP50, TP51, TP52, TP53, TP54, TP55, TP56, TP6, TP7, TP8, TP9: value TPPAD1-20 -> TPPAD1-13; device testpad:TPPAD1-20 -> testpad:TPPAD1-13
- U6: value 25Q40 -> ESP8266EX; device wifi:25Q40 -> wifi:ESP8266EX; PARTNO 25Q40 -> ESP8266EX
- U7: value ESP8266EX -> 25Q40; device wifi:ESP8266EX -> wifi:25Q40; PARTNO ESP8266EX -> 25Q40
Connections:
- removed net N$118: C29.2, U7.VDD3P3/4, U7.VDD_RTC/5
- removed net N$61 (its old number): DS7.G, R31.2
- new net N$59: DS13.G, R46.2
- net !CS: now also TP42.TP; no longer TP44.TP
- net !RESET0: now also TP37.TP; no longer TP39.TP
- net !RESET1: now also TP38.TP; no longer TP40.TP
- net 3.3V: now also C17.2, C18.1, C21.2, C22.1, C26.2, C27.1, C28.1, C29.1, C6.1, R12.2, R14.1, R36.2, R53.2, R9.1, U6.VDD3P3/3, U6.VDD3P3/4, U6.VDDA/1, U6.VDDA/30, U6.VDDD/29, U6.VDDPST/11, U6.VDDPST/17, U7.VCC; no longer C1.1, C16.2, C17.1, C19.1, C21.1, C25.2, C27.2, C28.2, C32.1, C33.1, C34.1, C35.1, R1.1, R12.1, R13.2, R20.2, R54.2, U6.VCC, U7.VDD3P3/3, U7.VDDA/1, U7.VDDA/30, U7.VDDD/29, U7.VDDPST/11, U7.VDDPST/17
- net CE: now also TP56.TP; no longer TP58.TP
- net CHIP_EN: now also TP48.TP, U6.CHIP_EN/7; no longer TP50.TP, U7.CHIP_EN/7
- net CLK: now also R57.1, U7.CLK; no longer R55.1, U6.CLK
- net CS: now also U6.SD_CMD/20, U7.CS#; no longer U6.CS#, U7.SD_CMD/20
- net CSN: now also TP55.TP, U1.PTD0/SPI0_PCS0; no longer TP57.TP, U1.PTC4/SPI0_PCS0
- net DIO: now also U6.SD_DATA_1/23, U7.DIO; no longer U6.DIO, U7.SD_DATA_1/23
- net DO: now also U6.SD_DATA_0/22, U7.DO; no longer U6.DO, U7.SD_DATA_0/22
- net FSYNC: now also TP39.TP; no longer TP41.TP
- net GND: now also C17.1, C18.2, C21.1, C25.2, C26.1, C27.2, C28.2, C29.2, C6.2, R13.1, R3.1, R31.2, R32.2, R33.2, R34.2, R35.2, R54.2, R55.1, R59.2, U6.PGND; no longer C1.2, C17.2, C18.1, C19.2, C21.2, C25.1, C27.1, C28.1, C29.1, C38.2, C39.2, C40.2, C41.2, R14.1, R15.2, R16.2, R17.2, R18.2, R19.2, R53.2, R57.1, R58.2, R9.1, U6.GND
- net GPIO0: now also TP50.TP, U6.GPIO0/15; no longer TP52.TP, U7.GPIO0/15
- net GPIO2: now also TP49.TP, U6.GPIO2/14; no longer TP51.TP, U7.GPIO2/14
- net HOLD#: now also U6.SD_DATA_2/18, U7.HOLD#; no longer U6.HOLD#, U7.SD_DATA_2/18
- net INT: now also TP43.TP; no longer TP45.TP
- net IRQ: now also TP51.TP; no longer TP53.TP
- net MISO: now also TP52.TP, U1.PTD3/SPI0_SIN; no longer TP54.TP, U1.PTC7/SPI0_SIN
- net MOSI: now also TP53.TP, U1.PTD2/SPI0_SOUT; no longer TP55.TP, U1.PTC6/SPI0_SOUT
- net N$100: now also C24.1, U6.XTAL_IN/28; no longer C22.1, U7.XTAL_IN/28
- net N$101: now also C19.1; no longer C26.1
- net N$102: now also R55.2, U6.MTCK/12; no longer R56.2, U7.MTCK/12
- net N$103: now also R56.2, U6.MTDO/13; no longer R57.2, U7.MTDO/13
- net N$107: now also R54.1, U6.RES12K/31; no longer R53.1, U7.RES12K/31
- net N$108: now also C32.1, R58.1; no longer C40.1, R59.1
- net N$109: now also C33.1, R58.2; no longer C41.1, R59.2
- net N$11: now also U1.PTC5/SPI0_SCK; no longer U1.PTD1/SPI0_SCK
- net N$111: now also L8.1; no longer L7.1
- net N$112: now also R59.1; no longer R58.1
- net N$114: now also L7.1; no longer L8.1
- net N$115: now also C37.1; no longer C39.1
- net N$116: now also L8.2; no longer L7.2
- net N$117: now also C34.1, C35.1, L7.2; no longer C37.1, C38.1, L8.2
- net N$15: now also U1.PTC4/SPI0_PCS0; no longer U1.PTD0/SPI0_PCS0
- net N$22: now also C19.2, U6.LNA/2; no longer C26.2, U7.LNA/2
- net N$23: now also C25.1, U6.XTAL_OUT/27; no longer C24.1, U7.XTAL_OUT/27
- net N$27: now also R12.1, R13.2; no longer R13.1, R14.2
- net N$28: now also R14.2; no longer R12.2
- net N$29: now also R7.2; no longer R2.2
- net N$3: now also R57.2, U6.SD_CLK/21; no longer R55.2, U7.SD_CLK/21
- net N$30: now also R32.1; no longer R16.1
- net N$31: now also R33.1; no longer R17.1
- net N$32: now also R34.1; no longer R18.1
- net N$33: now also R35.1; no longer R19.1
- net N$34: now also R36.1; no longer R20.1
- net N$35: now also R31.1; no longer R15.1
- net N$36: now also DS8.R, R27.2; no longer DS12.R, R44.2
- net N$37: now also DS7.R, R24.2; no longer DS10.R, R39.2
- net N$38: now also DS7.B, R25.2; no longer DS10.B, R40.2
- net N$39: now also DS7.G, R23.2; no longer DS10.G, R37.2
- net N$4: now also C16.2; no longer C18.2
- net N$40: now also DS8.B, R28.2; no longer DS12.B, R46.2
- net N$41: now also DS8.G, R26.2; no longer DS12.G, R42.2
- net N$42: now also DS10.G, R38.2; no longer DS5.G, R25.2
- net N$43: now also DS10.B, R37.2; no longer DS5.B, R22.2
- net N$44: now also DS9.B, R30.2; no longer DS14.B, R51.2
- net N$45: now also DS9.G, R29.2; no longer DS14.G, R48.2
- net N$46: now also R15.1; no longer R21.1
- net N$47: now also DS5.R, R19.2; no longer DS6.R, R28.2
- net N$48: now also R16.1; no longer R23.1
- net N$49: now also R17.1; no longer R24.1
- net N$5: now also U1.PTC7/SPI0_SIN; no longer U1.PTD3/SPI0_SIN
- net N$50: now also DS14.B, R47.2; no longer DS13.B, R43.2
- net N$51: now also R16.2; no longer R23.2
- net N$52: now also DS11.R, R40.2; no longer DS7.R, R29.2
- net N$53: now also R17.2; no longer R24.2
- net N$54: now also R15.2; no longer R21.2
- net N$55: now also DS5.B, R20.2; no longer DS6.B, R30.2
- net N$56: now also DS5.G, R18.2; no longer DS6.G, R26.2
- net N$58: now also DS12.B, R42.2; no longer DS9.B, R33.2
- net N$6: now also U1.PTC6/SPI0_SOUT; no longer U1.PTD2/SPI0_SOUT
- net N$60: now also R18.1; no longer R26.1
- net N$62: now also DS14.G, R49.2; no longer DS13.G, R47.2
- net N$63: now also DS11.B, R39.2; no longer DS7.B, R27.2
- net N$64: now also DS12.G, R44.2; no longer DS9.G, R36.2
- net N$65: now also DS6.B, R22.2; no longer DS8.B, R35.2
- net N$66: now also DS6.G, R21.2; no longer DS8.G, R32.2
- net N$67: now also DS14.R, R48.2; no longer DS13.R, R45.2
- net N$68: now also DS13.B, R45.2; no longer DS11.B, R38.2
- net N$69: now also R19.1; no longer R28.1
- net N$7: now also R6.2; no longer R1.2
- net N$70: now also R50.2; no longer R49.2
- net N$71: now also R20.1; no longer R30.1
- net N$72: now also R21.1; no longer R32.1
- net N$73: now also R22.1; no longer R35.1
- net N$74: now also R23.1; no longer R37.1
- net N$75: now also R24.1; no longer R39.1
- net N$76: now also R25.1; no longer R40.1
- net N$77: now also R26.1; no longer R42.1
- net N$78: now also R27.1; no longer R44.1
- net N$79: now also R28.1; no longer R46.1
- net N$80: now also R29.1; no longer R48.1
- net N$81: now also R30.1; no longer R51.1
- net N$82: now also DS12.R, R43.2; no longer DS9.R, R34.2
- net N$83: now also R51.2; no longer R50.2
- net N$84: now also R37.1; no longer R22.1
- net N$85: now also R38.1; no longer R25.1
- net N$86: now also R39.1; no longer R27.1
- net N$87: now also R40.1; no longer R29.1
- net N$88: now also R41.1; no longer R31.1
- net N$89: now also R42.1; no longer R33.1
- net N$90: now also R43.1; no longer R34.1
- net N$91: now also R44.1; no longer R36.1
- net N$92: now also R45.1; no longer R38.1
- net N$93: now also R46.1; no longer R41.1
- net N$94: now also R47.1; no longer R43.1
- net N$95: now also R48.1; no longer R45.1
- net N$96: now also R49.1; no longer R47.1
- net N$97: now also R50.1; no longer R49.1
- net N$98: now also R51.1; no longer R50.1
- net PTA0: now also R3.2; no longer R9.2
- net PTA1: now also R4.2; no longer R7.2
- net PTA3: now also R2.2; no longer R6.2
- net RESET_B: now also R5.2; no longer R8.2
- net SCK: now also TP54.TP, U1.PTD1/SPI0_SCK; no longer TP56.TP, U1.PTC5/SPI0_SCK
- net SCL: now also R9.2, TP40.TP; no longer R5.2, TP42.TP
- net SDA: now also R8.2, TP41.TP; no longer R4.2, TP37.TP, TP38.TP, TP43.TP
- net U0RX: now also TP45.TP, U6.U0RXD/25; no longer TP47.TP, U7.U0RXD/25
- net U0TX: now also TP44.TP, U6.U0TXD/26; no longer TP46.TP, U7.U0TXD/26
- net VDDA: now also C1.1, R1.1; no longer C5.1, R3.1
- net VREFH: now also C5.1, R1.2; no longer C6.1, R3.2
- net VREFL: now also C1.2; no longer C6.2
- net WIFI_RESET: now also R53.1, TP46.TP, U6.EXT_RSTB/32; no longer R54.1, TP48.TP, U7.EXT_RSTB/32
- net WP#: now also U6.SD_DATA_3/19, U7.WP#; no longer U6.WP#, U7.SD_DATA_3/19
- net XPD_DCDC: now also TP47.TP, U6.XPD_DCDC/8; no longer TP49.TP, U7.XPD_DCDC/8
Other:
- note added: "1: Y+ Group"
- note added: "2: X+ Group"
- note added: "3: Y- Group"
- note removed: "1: X+ Group"
- note removed: "2: Y- Group"
- note removed: "3: Y+ Group"
- moved on the sheet: C1, C16, C17, C18, C19, C2, C20, C21, C22, C23, C24, C25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

Commit message: More work on PCB.
Parts:
- removed C15: 10uF, SparkFun-Capacitors:CAP0603-CAP
- removed C16: 0.1 uF, SparkFun-Capacitors:CAP0402-CAP
- removed C37: 1.0 pF, SparkFun-Capacitors:CAP0402-CAP
- removed R30: 86.6, appfruits:RESISTOR0402
- removed R31, R32, R33, R34, R35: 10k, appfruits:RESISTOR0402
- removed R59: 22k, appfruits:RESISTOR0402
- C10: value 22uF -> 0.1uF; device SparkFun-Capacitors:CAP1210 -> SparkFun-Capacitors:CAP0402-CAP; PARTNO C3225X7R1A226K230AC -> C1005X7R1C104K050BC
- C12: value 0.1uF -> 22uF; device SparkFun-Capacitors:CAP0402-CAP -> SparkFun-Capacitors:CAP1210; PARTNO C1005X7R1C104K050BC -> C3225X7R1A226K230AC
- C14, C6, C8: value 10uF -> 0.1uF; device SparkFun-Capacitors:CAP0603-CAP -> SparkFun-Capacitors:CAP0402-CAP; PARTNO C1608X7S0J106M080AC -> C1005X7R1C104K050BC
- C19: value 5.6 pF -> 0.1 uF; PARTNO GRM1555C1H5R6CA01D -> C1005X7R1C104K050BC
- C20: value 10uF -> 5.6 pF; device SparkFun-Capacitors:CAP0603-CAP -> SparkFun-Capacitors:CAP0402-CAP; PARTNO C1608X7S0J106M080AC -> GRM1555C1H5R6CA01D
- C21, C29: value 0.1 uF -> 10uF; device SparkFun-Capacitors:CAP0402-CAP -> SparkFun-Capacitors:CAP0603-CAP; PARTNO C1005X7R1C104K050BC -> C1608X7S0J106M080AC
- C23, C27: value 10uF -> 0.1 uF; device SparkFun-Capacitors:CAP0603-CAP -> SparkFun-Capacitors:CAP0402-CAP; PARTNO C1608X7S0J106M080AC -> C1005X7R1C104K050BC
- C24: value 15 pF -> 10uF; device SparkFun-Capacitors:CAP0402-CAP -> SparkFun-Capacitors:CAP0603-CAP; PARTNO C1005C0G1H150J050BA -> C1608X7S0J106M080AC
- C26: value 0.1 uF -> 15 pF; PARTNO C1005X7R1C104K050BC -> C1005C0G1H150J050BA
- C30: value 10uF -> .033 uF; device SparkFun-Capacitors:CAP0603-CAP -> SparkFun-Capacitors:CAP0402-CAP; PARTNO C1608X7S0J106M080AC -> C1005X7R1H333K050BB
- C31: value .033 uF -> 22 pF; PARTNO C1005X7R1H333K050BB -> C1005C0G1H220J050BA
- C33: value 22 pF -> 2200 pF; PARTNO C1005C0G1H220J050BA -> C1005X7R1H222K050BA
- C34: value 2200 pF -> 4.7 pF; PARTNO C1005X7R1H222K050BA -> CGA2B2C0G1H4R7C050BA
- C35: value 4.7 pF -> 1.5 pF; PARTNO CGA2B2C0G1H4R7C050BA -> C1005C0G1H1R5B050BA
- C36: value 1.5 pF -> 1.0 pF; PARTNO C1005C0G1H1R5B050BA -> C1005C0G1H010B050BA
- C4, C7, C9: value 0.1uF -> 10uF; device SparkFun-Capacitors:CAP0402-CAP -> SparkFun-Capacitors:CAP0603-CAP; PARTNO C1005X7R1C104K050BC -> C1608X7S0J106M080AC
- R1: value 470 -> 10k; PARTNO CRCW0402470RFKED -> CRCW040210K0FKED
- R10: value 2M -> 220K; PARTNO CRCW04022M00FKED -> CRCW0402220KFKED
- R11: value 220K -> 1.2M; PARTNO CRCW0402220KFKED -> CRCW04021M20FKED
- R12: value 1.2M -> 220K; PARTNO CRCW04021M20FKED -> CRCW0402220KFKED
- R13: value 220K -> 25; PARTNO CRCW0402220KFKED -> CRCW040224R9FKED
- R14: value 25 -> 86.6; PARTNO CRCW040224R9FKED -> 5-1879213-0
- R36: value 10k -> 86.6; PARTNO CRCW040210K0FKED -> 5-1879213-0
- R5: value 10k -> 25; PARTNO CRCW040210K0FKED -> CRCW040224R9FKED
- R52: value 86.6 -> 12k; PARTNO 5-1879213-0 -> CRCW040212K0FKED
- R55: value 12k -> 10k; PARTNO CRCW040212K0FKED -> CRCW040210K0FKED
- R56: value 10k -> 200; PARTNO CRCW040210K0FKED -> CRCW0402200RFKED
- R57: value 200 -> 1M; PARTNO CRCW0402200RFKED -> CRCW04021M00FKED
- R58: value 1M -> 22k; PARTNO CRCW04021M00FKED -> CRCW040222K0FKED
- R7: value 25 -> 10k; PARTNO CRCW040224R9FKED -> CRCW040210K0FKED
- R9: value 10k -> 2M; PARTNO CRCW040210K0FKED -> CRCW04022M00FKED
- TP37, TP38, TP39, TP40, TP42, TP43, TP44, TP45, TP46, TP47, TP48, TP49, TP50, TP51, TP52, TP53, TP54, TP55, TP56: value TPPAD1-13 -> TPTP08R; device testpad:TPPAD1-13 -> testpad:TPTP08R
Connections:
- removed net N$30: R32.1, U3.A1
- removed net N$31: R33.1, U3.A0
- removed net N$32: R34.1, U4.A2
- removed net N$33: R35.1, U4.A1
- removed net N$34: R36.1, U4.A0
- removed net N$35: R31.1, U3.A2
- removed net VREFH: C5.1, R1.2, U1.VREFH
- removed net VREFL: C1.2, C5.2, C7.2, L2.2, U1.VREFL, U1.VSSA
- new net AGND: C4.2, C6.2, C8.2, L2.2, U1.VREFL, U1.VSSA
- net !RESET0: now also TP39.TP; no longer TP37.TP
- net !RESET1: now also TP40.TP; no longer TP38.TP
- net 3.3V: now also C1.1, C18.2, C19.1, C21.1, C22.2, C24.1, C5.1, C7.1, R1.1, R11.2, R13.1, R3.1, R52.2, TP1.TP, TP16.TP, TP17.TP, TP2.TP, TP32.TP, TP33.TP, TP34.TP, TP35.TP, U4.A0; no longer C10.1, C15.1, C17.2, C18.1, C20.1, C21.2, C22.1, C26.2, C30.1, C4.1, C6.1, R12.2, R14.1, R2.1, R36.2, R53.2, R9.1, TP12.TP, TP15.TP, TP19.TP, TP24.TP, TP25.TP, TP30.TP, TP6.TP, TP9.TP
- net CHIP_EN: now also TP46.TP; no longer TP48.TP
- net CLK: now also R56.1; no longer R57.1
- net FSYNC: now also TP41.TP; no longer TP39.TP
- net GND: now also C1.2, C18.1, C19.2, C21.2, C22.1, C26.2, C30.1, C31.2, C36.2, C5.2, C7.2, R10.1, R12.1, R2.1, R53.2, R54.1, R58.2, TP13.TP, TP15.TP, TP25.TP, TP27.TP, TP28.TP, TP30.TP, TP4.TP, TP6.TP, U3.A0, U3.A1, U3.A2, U4.A1, U4.A2; no longer C15.2, C16.1, C18.2, C20.2, C21.1, C22.2, C26.1, C30.2, C31.1, C35.2, C37.2, C4.2, C6.2, C8.2, R11.1, R13.1, R3.1, R31.2, R32.2, R33.2, R34.2, R35.2, R54.2, R56.1, R59.2, TP11.TP, TP17.TP, TP2.TP, TP20.TP, TP23.TP, TP32.TP, TP35.TP, TP8.TP
- net GPIO0: now also TP49.TP; no longer TP50.TP
- net GPIO2: now also TP47.TP; no longer TP49.TP
- net N$100: now also C25.1; no longer C24.1
- net N$101: now also C20.1; no longer C19.1
- net N$102: now also R54.2; no longer R55.2
- net N$103: now also R55.2; no longer R56.2
- net N$107: now also R53.1; no longer R54.1
- net N$108: now also C31.1, R57.1; no longer C32.1, R58.1
- net N$109: now also C32.1, R57.2; no longer C33.1, R58.2
- net N$11: now also TP9.TP; no longer TP33.TP
- net N$112: now also R58.1; no longer R59.1
- net N$113: now also C30.2; no longer C31.2
- net N$115: now also C35.2, C36.1; no longer C36.2, C37.1
- net N$116: now also C35.1; no longer C36.1
- net N$117: now also C33.1; no longer C35.1
- net N$12: now also TP10.TP; no longer TP22.TP
- net N$14: now also TP11.TP; no longer TP28.TP
- net N$15: now also TP12.TP; no longer TP34.TP
- net N$16: now also TP24.TP; no longer TP16.TP
- net N$17: now also TP21.TP; no longer TP7.TP
- net N$18: now also TP22.TP; no longer TP10.TP
- net N$19: now also TP23.TP; no longer TP13.TP
- net N$20: now also TP20.TP; no longer TP4.TP
- net N$21: now also TP19.TP; no longer TP1.TP
- net N$22: now also C20.2; no longer C19.2
- net N$23: now also C26.1; no longer C25.1
- net N$25: now also C10.1; no longer C9.1
- net N$26: now also R10.2, R9.1; no longer R10.1, R11.2
- net N$27: now also R11.1, R12.2; no longer R12.1, R13.2
- net N$28: now also R13.2; no longer R14.2
- net N$29: now also R6.2; no longer R7.2
- net N$3: now also R56.2; no longer R57.2
- net N$36: now also R26.2; no longer R27.2
- net N$37: now also R23.2; no longer R24.2
- net N$38: now also R24.2; no longer R25.2
- net N$39: now also R22.2; no longer R23.2
- net N$4: now also C17.2; no longer C16.2
- net N$40: now also R27.2; no longer R28.2
- net N$41: now also R25.2; no longer R26.2
- net N$42: now also R37.2; no longer R38.2
- net N$43: now also R36.2; no longer R37.2
- net N$44: now also R29.2; no longer R30.2
- net N$45: now also R28.2; no longer R29.2
- net N$46: now also R14.1; no longer R15.1
- net N$47: now also R18.2; no longer R19.2
- net N$48: now also R15.1; no longer R16.1
- net N$49: now also R16.1; no longer R17.1
- net N$5: now also TP7.TP; no longer TP21.TP
- net N$50: now also R46.2; no longer R47.2
- net N$51: now also R15.2; no longer R16.2
- net N$52: now also R39.2; no longer R40.2
- net N$53: now also R16.2; no longer R17.2
- net N$54: now also R14.2; no longer R15.2
- net N$55: now also R19.2; no longer R20.2
- net N$56: now also R17.2; no longer R18.2
- net N$57: now also R51.2; no longer R52.2
- net N$58: now also R41.2; no longer R42.2
- net N$59: now also R45.2; no longer R46.2
- net N$6: now also TP8.TP; no longer TP27.TP
- net N$60: now also R17.1; no longer R18.1
- net N$61: now also R40.2; no longer R41.2
- net N$62: now also R48.2; no longer R49.2
- net N$63: now also R38.2; no longer R39.2
- net N$64: now also R43.2; no longer R44.2
- net N$65: now also R21.2; no longer R22.2
- net N$66: now also R20.2; no longer R21.2
- net N$67: now also R47.2; no longer R48.2
- net N$68: now also R44.2; no longer R45.2
- net N$69: now also R18.1; no longer R19.1
- net N$7: now also R5.2; no longer R6.2
- net N$70: now also R49.2; no longer R50.2
- net N$71: now also R19.1; no longer R20.1
- net N$72: now also R20.1; no longer R21.1
- net N$73: now also R21.1; no longer R22.1
- net N$74: now also R22.1; no longer R23.1
- net N$75: now also R23.1; no longer R24.1
- net N$76: now also R24.1; no longer R25.1
- net N$77: now also R25.1; no longer R26.1
- net N$78: now also R26.1; no longer R27.1
- net N$79: now also R27.1; no longer R28.1
- net N$80: now also R28.1; no longer R29.1
- net N$81: now also R29.1; no longer R30.1
- net N$82: now also R42.2; no longer R43.2
- net N$83: now also R50.2; no longer R51.2
- net N$84: now also R36.1; no longer R37.1
- net N$85: now also R37.1; no longer R38.1
- net N$86: now also R38.1; no longer R39.1
- net N$87: now also R39.1; no longer R40.1
- net N$88: now also R40.1; no longer R41.1
- net N$89: now also R41.1; no longer R42.1
- net N$90: now also R42.1; no longer R43.1
- net N$91: now also R43.1; no longer R44.1
- net N$92: now also R44.1; no longer R45.1
- net N$93: now also R45.1; no longer R46.1
- net N$94: now also R46.1; no longer R47.1
- net N$95: now also R47.1; no longer R48.1
- net N$96: now also R48.1; no longer R49.1
- net N$97: now also R49.1; no longer R50.1
- net N$98: now also R50.1; no longer R51.1
- net N$99: now also R51.1; no longer R52.1
- net PTA0: now also R2.2; no longer R3.2
- net PTA1: now also R3.2; no longer R4.2
- net PTA3: now also R1.2; no longer R2.2
- net RESET_B: now also R4.2; no longer R5.2
- net SCL: now also R8.2, TP38.TP; no longer R9.2, TP40.TP
- net SDA: now also R7.2, TP37.TP; no longer R8.2, TP41.TP
- net U0RX: now also TP50.TP; no longer TP45.TP
- net U0TX: now also TP48.TP; no longer TP44.TP
- net VDDA: now also C4.1, C6.1, U1.VREFH; no longer C1.1, R1.1
- net VREF_OUT: now also C8.1; no longer C7.1
- net V_IN: now also C9.1, R9.2; no longer C8.1, R10.2
- net WIFI_RESET: now also R52.1, TP45.TP; no longer R53.1, TP46.TP
- net XPD_DCDC: now also TP44.TP; no longer TP47.TP
Other:
- moved on the sheet: C1, C10, C11, C13, C14, C17, C18, C2, C20, C21, C22, C23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

Commit message: More board layout. Renumbered x+ and y+ to match what I did on the PCB.
Parts:
- removed C35: 1.5 pF, SparkFun-Capacitors:CAP0402-CAP
- removed C36: 1.0 pF, SparkFun-Capacitors:CAP0402-CAP
- removed L8: 3.9 nH, SparkFun-Passives:INDUCTOR0402
- removed R53, R54: 12k, appfruits:RESISTOR0402
- removed R55: 10k, appfruits:RESISTOR0402
- removed R56: 200, appfruits:RESISTOR0402
- removed R57: 1M, appfruits:RESISTOR0402
- removed R58: 22k, appfruits:RESISTOR0402
- added C15, C16: 0.1 uF, SparkFun-Capacitors:CAP0402-CAP
- added R30, R31, R32, R33, R34, R35: 86.6, appfruits:RESISTOR0402
- C18: value 0.1 uF -> 5.6 pF; PARTNO C1005X7R1C104K050BC -> GRM1555C1H5R6CA01D
- C19, C22, C27: value 0.1 uF -> 10uF; device SparkFun-Capacitors:CAP0402-CAP -> SparkFun-Capacitors:CAP0603-CAP; PARTNO C1005X7R1C104K050BC -> C1608X7S0J106M080AC
- C20: value 5.6 pF -> 0.1 uF; PARTNO GRM1555C1H5R6CA01D -> C1005X7R1C104K050BC
- C21: value 10uF -> 0.1 uF; device SparkFun-Capacitors:CAP0603-CAP -> SparkFun-Capacitors:CAP0402-CAP; PARTNO C1608X7S0J106M080AC -> C1005X7R1C104K050BC
- C23: value 0.1 uF -> 15 pF; PARTNO C1005X7R1C104K050BC -> C1005C0G1H150J050BA
- C24: value 10uF -> 15 pF; device SparkFun-Capacitors:CAP0603-CAP -> SparkFun-Capacitors:CAP0402-CAP; PARTNO C1608X7S0J106M080AC -> C1005C0G1H150J050BA
- C25, C26: value 15 pF -> 0.1 uF; PARTNO C1005C0G1H150J050BA -> C1005X7R1C104K050BC
- C28: value 0.1 uF -> .033 uF; PARTNO C1005X7R1C104K050BC -> C1005X7R1H333K050BB
- C29: value 10uF -> 22 pF; device SparkFun-Capacitors:CAP0603-CAP -> SparkFun-Capacitors:CAP0402-CAP; PARTNO C1608X7S0J106M080AC -> C1005C0G1H220J050BA
- C30: value .033 uF -> 22 pF; PARTNO C1005X7R1H333K050BB -> C1005C0G1H220J050BA
- C31: value 22 pF -> 2200 pF; PARTNO C1005C0G1H220J050BA -> C1005X7R1H222K050BA
- C32: value 22 pF -> 4.7 pF; PARTNO C1005C0G1H220J050BA -> CGA2B2C0G1H4R7C050BA
- C33: value 2200 pF -> 1.5 pF; PARTNO C1005X7R1H222K050BA -> C1005C0G1H1R5B050BA
- C34: value 4.7 pF -> 1.0 pF; PARTNO CGA2B2C0G1H4R7C050BA -> C1005C0G1H010B050BA
- C4, C7: value 10uF -> 0.1uF; device SparkFun-Capacitors:CAP0603-CAP -> SparkFun-Capacitors:CAP0402-CAP; PARTNO C1608X7S0J106M080AC -> C1005X7R1C104K050BC
- C5, C6: value 0.1uF -> 10uF; device SparkFun-Capacitors:CAP0402-CAP -> SparkFun-Capacitors:CAP0603-CAP; PARTNO C1005X7R1C104K050BC -> C1608X7S0J106M080AC
- L2: value 600 Ohm/100 Mhz -> 2.2uH, 1.4A; device appfruits:INDUCTOR-BK2125HM601-T -> appfruits:LPS30152.2UH; PARTNO BK2125HM601-T -> BRL3225T2R2M
- L3: value 2.2uH, 1.4A -> DNP; device appfruits:LPS30152.2UH -> SparkFun-Passives:INDUCTOR30OHM,1.8A; PARTNO BRL3225T2R2M -> DNP
- L5: value DNP -> 8.2 nH; device SparkFun-Passives:INDUCTOR30OHM,1.8A -> SparkFun-Passives:INDUCTOR0402; PARTNO DNP -> L-07C8N2JV6T
- L6: value 8.2 nH -> 2.7 nH; PARTNO L-07C8N2JV6T -> L-07C2N7SV6T
- L7: value 2.7 nH -> 3.9 nH; PARTNO L-07C2N7SV6T -> L-07C3N9SV6T
- R46, R47, R48: value 86.6 -> 12k; PARTNO 5-1879213-0 -> CRCW040212K0FKED
- R49: value 86.6 -> 10k; PARTNO 5-1879213-0 -> CRCW040210K0FKED
- R50: value 86.6 -> 200; PARTNO 5-1879213-0 -> CRCW0402200RFKED
- R51: value 86.6 -> 1M; PARTNO 5-1879213-0 -> CRCW04021M00FKED
- R52: value 12k -> 22k; PARTNO CRCW040212K0FKED -> CRCW040222K0FKED
- TP41: value TPPAD1-13 -> TPTP08R; device testpad:TPPAD1-13 -> testpad:TPTP08R
Connections:
- removed net AGND: C4.2, C6.2, C8.2, L2.2, U1.VREFL, U1.VSSA
- net !CS: now also U1.PTC4/SPI0_PCS0; no longer U1.PTC2/ADC0_SE12
- net !RESET0: now also U1.PTC10/ADC1_SE6B; no longer U1.PTA4
- net 3.3V: now also C16.2, C17.1, C20.2, C22.1, C25.1, C26.1, C4.1, R46.2; no longer C18.2, C22.2, C23.1, C24.1, C28.1, C29.1, C7.1, R52.2
- net CE: now also U1.PTD7/UART0_TX; no longer U1.PTC9/ADC1_SE5B
- net CLK: now also R50.1; no longer R56.1
- net CSN: now also U1.PTD6/UART0_RX; no longer U1.PTD0/SPI0_PCS0
- net FSYNC: now also U1.PTC11/ADC1_SE7B; no longer U1.PTB1/ADC0_SE9
- net GND: now also C15.1, C16.1, C17.2, C20.1, C22.2, C28.1, C30.2, C4.2, C6.2, C8.2, L3.2, R47.2, R48.1, R49.1, R52.2, U1.VREFL, U1.VSSA; no longer C17.1, C18.1, C22.1, C28.2, C30.1, C33.2, C36.2, L2.1, L5.2, R53.2, R54.1, R55.1, R58.2
- net INT: now also U1.PTC9/ADC1_SE5B; no longer U1.PTB0/ADC0_SE8
- net N$10: now also U1.PTD0/SPI0_PCS0; no longer U1.PTD6/UART0_RX
- net N$100: now also C23.1; no longer C25.1
- net N$101: now also C18.1, L3.1; no longer C20.1, L4.1
- net N$102: now also R48.2; no longer R54.2
- net N$103: now also R49.2; no longer R55.2
- net N$107: now also R47.1; no longer R53.1
- net N$108: now also C29.1, R51.1; no longer C31.1, R57.1
- net N$109: now also C30.1, R51.2; no longer C32.1, R57.2
- net N$111: now also L5.1, L7.1; no longer L6.1, L8.1
- net N$112: now also R52.1; no longer R58.1
- net N$113: now also C28.2; no longer C30.2
- net N$114: now also L5.2, L6.1; no longer L6.2, L7.1
- net N$115: now also C33.2, C34.1; no longer C35.2, C36.1
- net N$116: now also C33.1, L7.2; no longer C35.1, L8.2
- net N$117: now also C31.1, C32.1, L6.2; no longer C33.1, C34.1, L7.2
- net N$12: now also U1.PTC2/SPI0_PCS2; no longer U1.PTD5/SPI0_PCS2
- net N$13: now also U1.PTD4/SPI0_PCS1; no longer U1.PTD7/UART0_TX
- net N$14: now also U1.PTB1/ADC0_SE9; no longer U1.PTD4/SPI0_PCS1
- net N$15: now also U1.PTB0/ADC0_SE8; no longer U1.PTC4/SPI0_PCS0
- net N$16: now also U1.PTD5/SPI0_PCS2; no longer U1.PTC11/ADC1_SE7B
- net N$17: now also U1.PTA4; no longer U1.PTC10/ADC1_SE6B
- net N$18: now also U1.PTE1/I2C1_SCL/UART1_RX; no longer U1.PTE0/I2C1_SDA/UART1_TX
- net N$19: now also U1.PTE0/I2C1_SDA/UART1_TX; no longer U1.PTE1/I2C1_SCL/UART1_RX
- net N$22: now also C18.2, L4.1; no longer C20.2, L5.1
- net N$23: now also C24.1; no longer C26.1
- net N$24: now also L2.1; no longer L3.1
- net N$3: now also R50.2; no longer R56.2
- net N$4: now also C15.2; no longer C17.2
- net N$42: now also R31.2; no longer R37.2
- net N$43: now also R30.2; no longer R36.2
- net N$50: now also R40.2; no longer R46.2
- net N$52: now also R33.2; no longer R39.2
- net N$57: now also R45.2; no longer R51.2
- net N$58: now also R35.2; no longer R41.2
- net N$59: now also R39.2; no longer R45.2
- net N$61: now also R34.2; no longer R40.2
- net N$62: now also R42.2; no longer R48.2
- net N$63: now also R32.2; no longer R38.2
- net N$64: now also R37.2; no longer R43.2
- net N$67: now also R41.2; no longer R47.2
- net N$68: now also R38.2; no longer R44.2
- net N$70: now also R43.2; no longer R49.2
- net N$82: now also R36.2; no longer R42.2
- net N$83: now also R44.2; no longer R50.2
- net N$84: now also R30.1; no longer R36.1
- net N$85: now also R31.1; no longer R37.1
- net N$86: now also R32.1; no longer R38.1
- net N$87: now also R33.1; no longer R39.1
- net N$88: now also R34.1; no longer R40.1
- net N$89: now also R35.1; no longer R41.1
- net N$90: now also R36.1; no longer R42.1
- net N$91: now also R37.1; no longer R43.1
- net N$92: now also R38.1; no longer R44.1
- net N$93: now also R39.1; no longer R45.1
- net N$94: now also R40.1; no longer R46.1
- net N$95: now also R41.1; no longer R47.1
- net N$96: now also R42.1; no longer R48.1
- net N$97: now also R43.1; no longer R49.1
- net N$98: now also R44.1; no longer R50.1
- net N$99: now also R45.1; no longer R51.1
- net VDDA: now also C7.1; no longer C4.1
- net V_IN: now also L2.2; no longer L3.2
- net WIFI_RESET: now also R46.1; no longer R52.1
Other:
- note added: "1: X+ Group"
- note added: "2: Y+ Group"
- note removed: "1: Y+ Group"
- note removed: "2: X+ Group"
- moved on the sheet: C17, C20, C21, C22, C23, C24, C27, C28, C29, C30, C31, C32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
