File: Circuit/P1R5/P1R5.brd (EAGLE design)
At the start: 160 x 100 mm, 165 parts, among them J1 2X5_0.05"_CORTEX_DEBUGTH_NOKE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, U1 MK20DX256VLH7, U102 TPS61200, U403 MPU-9250, Y1 16Mhz/8pF, Y2 32.768KHz, Y203 26 Mhz, Y304 16 Mhz

Commit message: More schematic cleanup.
Verified layouts, will probably check them again anyway.
Still need to do the passives and fix part numbers so they match the
bom-ex db.
Parts:
- removed C101: 10uF, appfruits:0603-CAP
- removed C102, C104, C501, C505: 0.1uF, appfruits:0603-CAP
- removed C103: 22uF, appfruits:0603-CAP
- removed C206: 5.6 pF, SparkFun-Capacitors:0603-CAP
- removed C207, C223: 15 pF, SparkFun-Capacitors:0603-CAP
- removed C222: 1 uF, SparkFun-Capacitors:0603-CAP
- removed C226, C228, C233, C234, C235, C336, C337, C424, C425, C427: .1 uF, SparkFun-Capacitors:0603-CAP
- removed C308: 33 nF, SparkFun-Capacitors:0603-CAP
- removed C309: 2.2 nF, SparkFun-Capacitors:0603-CAP
- removed C310: 4.7 pF, SparkFun-Capacitors:0603-CAP
- removed C312: 1.0 pF, SparkFun-Capacitors:0603-CAP
- removed C313: 1.5 pF, SparkFun-Capacitors:0603-CAP
- removed C314, C315: 22 pF, SparkFun-Capacitors:0603-CAP
- removed C502, C507: 2.2uF, appfruits:0603-CAP
- removed JP503: (no value), SparkFun:1X04
- removed L101: 2.2uH, 2.1A, appfruits:LPS3015
- removed L207, L208: DNP, SparkFun-Passives:0603
- removed L302: 2.7 nH, SparkFun-Passives:C0402
- removed L305: 8.2 nH, SparkFun-Passives:C0402
- removed L306: 3.9 nH, SparkFun-Passives:C0402
- removed LED101: (no value), appfruits:LED-0603
- removed R103: 2M, appfruits:0603-RES
- removed R104, R106: 220K, appfruits:0603-RES
- removed R107: 1.2M, appfruits:0603-RES
- removed R109: 470, appfruits:0603-RES
- removed R201, R205, R215: 12k, SparkFun-Resistors:0603-RES
- removed R218: 200, SparkFun-Resistors:0603-RES
- removed R251: 10k, SparkFun-Resistors:0603-RES
- removed R311: 1M, SparkFun-Resistors:0603-RES
- removed R312: 22k, SparkFun-Resistors:0603-RES
- removed R519, R520, R521, R522, R523, R524: 10k, SparkFun:0603-RES
- removed R525, R526, R527, R528, R529, R530, R531, R532, R533, R534, R535, R536, R537, R538, R539, R540, R541, R542, R543, R544, R545, R546, R547, R548: (no value), SparkFun:0402-RES
- removed U$201, U$302: ANTENNA2SMD, SparkFun-RF:ANTENNA-CHIP2
- removed U$203: 25Q40, wifi:SOP8
- removed U$206: ESP8266EX, wifi:QFN32
- removed U$304: NRF24L01, RF:QFN20(4X4)
- removed U$508, U$511, U$513, U$514, U$515, U$516, U$517, U$518: LTST-C19FD1WT, led:LTST-C19FD1WT
- removed U$520, U$521: PCA9552BS, NXP_By_element14_Batch_1:HVQFN24
- removed U102: TPS61200, appfruits:QFN-10_PAD
- removed U403: MPU-9250, chips:QFN-24/3MM
- removed Y203: 26 Mhz, SparkFun-FreqCtrl:CRYSTAL-SMD-5X3
- removed Y304: 16 Mhz, SparkFun-FreqCtrl:CRYSTAL-SMD-5X3
- added AE1, AE2: ANTENNA2SMD, SparkFun-RF:ANTENNA-CHIP2
- added C13, C15, C17, C19, C36: 0.1uF, appfruits:0603-CAP
- added C14: 10uF, appfruits:0603-CAP
- added C16: 22uF, appfruits:0603-CAP
- added C18, C20, C37: 2.2uF, appfruits:0603-CAP
- added C21, C22, C23, C24, C25, C28, C31, C32, C34, C35: .1 uF, SparkFun-Capacitors:0603-CAP
- added C26, C27: 15 pF, SparkFun-Capacitors:0603-CAP
- added C29: 5.6 pF, SparkFun-Capacitors:0603-CAP
- added C30: 1 uF, SparkFun-Capacitors:0603-CAP
- added C33: 33 nF, SparkFun-Capacitors:0603-CAP
- added C38: 1.5 pF, SparkFun-Capacitors:0603-CAP
- added C39: 2.2 nF, SparkFun-Capacitors:0603-CAP
- added C40: 4.7 pF, SparkFun-Capacitors:0603-CAP
- added C41: 1.0 pF, SparkFun-Capacitors:0603-CAP
- added C42, C43: 22 pF, SparkFun-Capacitors:0603-CAP
- added DS1, DS10, DS11, DS12, DS2, DS3, DS4, DS5, DS6, DS7, DS8, DS9: LTST-C19FD1WT, led:LTST-C19FD1WT
- added L3: 2.2uH, 1.4A, appfruits:LPS3015
- added L4, L5: DNP, SparkFun-Passives:0603
- added L6: 8.2 nH, SparkFun-Passives:C0402
- added L7: 3.9 nH, SparkFun-Passives:C0402
- added L8: 2.7 nH, SparkFun-Passives:C0402
- added LED3: (no value), appfruits:LED-0603
- added R10: 2M, appfruits:0603-RES
- added R11: 1.2M, appfruits:0603-RES
- added R12: 470, appfruits:0603-RES
- added R13, R14: 220K, appfruits:0603-RES
- added R15, R16, R17, R18, R19, R20: 10k, SparkFun:0603-RES
- added R21, R22, R23, R24, R25, R26, R27, R28, R29, R30, R31, R32, R33, R34, R35, R36, R37, R38, R39, R40, R41, R42, R43, R44, R45, R46, R47, R48, R49, R50, R51, R52: (no value), SparkFun:0402-RES
- added R53, R54, R56: 12k, SparkFun-Resistors:0603-RES
- added R55: 200, SparkFun-Resistors:0603-RES
- added R57: 10k, SparkFun-Resistors:0603-RES
- added R58: 22k, SparkFun-Resistors:0603-RES
- added R59: 1M, SparkFun-Resistors:0603-RES
- added U2: TPS61200, appfruits:QFN-10_PAD
- added U3, U4: PCA9552BS, NXP_By_element14_Batch_1:HVQFN24
- added U5: MPU-9250, chips:QFN-24/3MM
- added U6: 25Q40, wifi:SOP8
- added U7: ESP8266EX, wifi:QFN32
- added U8: NRF24L01, RF:QFN20(4X4)
- added Y3: 26 Mhz, SparkFun-FreqCtrl:CRYSTAL-SMD-5X3
- added Y4: 16 Mhz, SparkFun-FreqCtrl:CRYSTAL-SMD-5X3
- C1, C7: value 2.2uF -> 0.1uF
- C5, C6: value 0.1uF -> 2.2uF
- R2, R3: value (none) -> 470; device SparkFun:0402-RES -> appfruits:0603-RES
- R4, R5: value (none) -> 10k; device SparkFun:0402-RES -> SparkFun-Resistors:0603-RES
- R6, R7: value 470 -> (none); device appfruits:0603-RES -> SparkFun:0402-RES
- R8, R9: value 10k -> (none); device SparkFun-Resistors:0603-RES -> SparkFun:0402-RES
- moved TP35 158.8 mm to (-73.7, -105.4)
- moved TP29 133.4 mm to (-73.7, -111.8)
- moved TP2 127.0 mm to (-73.7, -238.8)
- moved TP3 120.8 mm to (-67.3, -238.8)
- moved TP6 108.0 mm to (-73.7, -245.1)
- moved TP23 108.0 mm to (-73.7, -118.1)
- moved TP24 101.8 mm to (-73.7, -124.5)
- moved TP28 101.8 mm to (-73.7, -137.2)
- moved TP5 101.8 mm to (-67.3, -232.4)
- moved TP33 101.6 mm to (-73.7, -156.2)
- moved TP34 95.5 mm to (-73.7, -162.6)
- moved TP22 89.1 mm to (-73.7, -130.8)
- moved TP9 89.1 mm to (-67.3, -245.1)
- moved TP27 88.9 mm to (-73.7, -149.9)
- moved TP8 82.5 mm to (-73.7, -232.4)
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Connections:
- removed net IMU1:N$4: C427.2, U403.10
- removed net LED_DRIVER1:N$1: R527.1, U$520.3
- removed net LED_DRIVER1:N$10: R535.1, U$520.11
- removed net LED_DRIVER1:N$11: R536.1, U$520.12
- removed net LED_DRIVER1:N$12: R534.1, U$520.13
- removed net LED_DRIVER1:N$13: JP503.4, U$520.14
- removed net LED_DRIVER1:N$14: R520.1, U$520.23
- removed net LED_DRIVER1:N$15: R521.1, U$520.22
- removed net LED_DRIVER1:N$16: R538.1, U$521.1
- removed net LED_DRIVER1:N$17: R539.1, U$521.2
- removed net LED_DRIVER1:N$18: R537.1, U$521.3
- removed net LED_DRIVER1:N$19: R541.1, U$521.4
- removed net LED_DRIVER1:N$2: R526.1, U$520.1
- removed net LED_DRIVER1:N$20: R542.1, U$521.5
- removed net LED_DRIVER1:N$21: R540.1, U$521.6
- removed net LED_DRIVER1:N$22: R544.1, U$521.7
- removed net LED_DRIVER1:N$23: R545.1, U$521.8
- removed net LED_DRIVER1:N$24: R543.1, U$521.10
- removed net LED_DRIVER1:N$25: R547.1, U$521.11
- removed net LED_DRIVER1:N$26: R548.1, U$521.12
- removed net LED_DRIVER1:N$27: R546.1, U$521.13
- removed net LED_DRIVER1:N$28: R524.1, U$521.24
- removed net LED_DRIVER1:N$29: R523.1, U$521.23
- removed net LED_DRIVER1:N$3: R528.1, U$520.6
- removed net LED_DRIVER1:N$30: R522.1, U$521.22
- removed net LED_DRIVER1:N$33: R519.1, U$520.24
- removed net LED_DRIVER1:N$37: JP503.2, U$520.16
- removed net LED_DRIVER1:N$38: JP503.1, U$520.17
- removed net LED_DRIVER1:N$39: JP503.3, U$520.15
- removed net LED_DRIVER1:N$4: R525.1, U$520.2
- removed net LED_DRIVER1:N$47: R529.2, U$511.R
- removed net LED_DRIVER1:N$48: R541.2, U$516.R
- removed net LED_DRIVER1:N$49: R547.2, U$518.R
- removed net LED_DRIVER1:N$5: R529.1, U$520.4
- removed net LED_DRIVER1:N$50: R543.2, U$517.B
- removed net LED_DRIVER1:N$51: R532.2, U$513.R
- removed net LED_DRIVER1:N$52: R535.2, U$514.R
- removed net LED_DRIVER1:N$53: R531.2, U$513.B
- removed net LED_DRIVER1:N$54: R533.2, U$513.G
- removed net LED_DRIVER1:N$55: R528.2, U$511.B
- removed net LED_DRIVER1:N$56: R530.2, U$511.G
- removed net LED_DRIVER1:N$57: R548.2, U$518.G
- removed net LED_DRIVER1:N$58: R537.2, U$515.B
- removed net LED_DRIVER1:N$59: R542.2, U$516.G
- removed net LED_DRIVER1:N$6: R530.1, U$520.5
- removed net LED_DRIVER1:N$60: R526.2, U$508.R
- removed net LED_DRIVER1:N$61: R536.2, U$514.G
- removed net LED_DRIVER1:N$62: R545.2, U$517.G
- removed net LED_DRIVER1:N$63: R534.2, U$514.B
- removed net LED_DRIVER1:N$64: R539.2, U$515.G
- removed net LED_DRIVER1:N$65: R527.2, U$508.B
- removed net LED_DRIVER1:N$66: R525.2, U$508.G
- removed net LED_DRIVER1:N$67: R544.2, U$517.R
- removed net LED_DRIVER1:N$68: R540.2, U$516.B
- removed net LED_DRIVER1:N$69: R538.2, U$515.R
- removed net LED_DRIVER1:N$7: R532.1, U$520.7
- removed net LED_DRIVER1:N$70: R546.2, U$518.B
- removed net LED_DRIVER1:N$8: R533.1, U$520.8
- removed net LED_DRIVER1:N$9: R531.1, U$520.10
- removed net MESH1:N$1: C309.1, C310.1, L302.2, U$304.11
- removed net MESH1:N$10: L305.1, L306.1, U$304.13
- removed net MESH1:N$11: R312.1, U$304.16
- removed net MESH1:N$12: C308.2, U$304.19
- removed net MESH1:N$13: L302.1, L305.2, U$304.12
- removed net MESH1:N$14: C312.1, C313.2, U$302.FEED
- removed net MESH1:N$24: C313.1, L306.2
- removed net MESH1:N$7: C314.1, R311.1, U$304.9, Y304.1
- removed net MESH1:N$8: C315.1, R311.2, U$304.10, Y304.3
- removed net VREG1:N$1: L101.1, U102.3
- removed net VREG1:N$2: C104.1, U102.1
- removed net VREG1:N$3: C102.2, R103.1, R104.2, U102.7
- removed net VREG1:N$4: R106.2, R107.1, U102.10
- removed net VREG1:N$5: LED101.A, R109.2
- removed net WIFI1:CLK: R218.1, U$203.6
- removed net WIFI1:CS: U$203.1, U$206.SD_CMD/20
- removed net WIFI1:DIO: U$203.5, U$206.SD_DATA_1/23
- removed net WIFI1:DO: U$203.2, U$206.SD_DATA_0/22
- removed net WIFI1:HOLD#: U$203.7, U$206.SD_DATA_2/18
- removed net WIFI1:N$11: C207.1, U$206.XTAL_OUT/27, Y203.1
- removed net WIFI1:N$12: C223.1, U$206.XTAL_IN/28, Y203.3
- removed net WIFI1:N$14: C206.1, L207.1, U$201.FEED
- removed net WIFI1:N$16: R205.2, U$206.MTCK/12
- removed net WIFI1:N$22: R251.2, U$206.MTDO/13
- removed net WIFI1:N$25: C233.2, U$206.VDDA/1
- removed net WIFI1:N$26: C226.2, U$206.VDD3P3/3
- removed net WIFI1:N$27: C228.2, U$206.VDD3P3/4
- removed net WIFI1:N$5: R218.2, U$206.SD_CLK/21
- removed net WIFI1:N$7: C206.2, L208.1, U$206.LNA/2
- removed net WIFI1:N$8: R201.1, U$206.RES12K/31
- removed net WIFI1:WP#: U$203.3, U$206.SD_DATA_3/19
- new net !CS: U1.45, U5.22
- new net !RESET0: U1.26, U3.18
- new net !RESET1: U1.27, U4.18
- new net CLK: R55.1, U6.6
- new net CS: U6.1, U7.SD_CMD/20
- new net DIO: U6.5, U7.SD_DATA_1/23
- new net DO: U6.2, U7.SD_DATA_0/22
- new net HOLD#: U6.7, U7.SD_DATA_2/18
- new net N$100: C26.1, U7.XTAL_IN/28, Y3.3
- new net N$101: AE1.FEED, C29.1, L4.1
- new net N$102: R56.2, U7.MTCK/12
- new net N$103: R57.2, U7.MTDO/13
- new net N$107: R53.1, U7.RES12K/31
- new net N$108: C42.1, R59.1, U8.9, Y4.1
- new net N$109: C43.1, R59.2, U8.10, Y4.3
- new net N$111: L6.1, L7.1, U8.13
- new net N$112: R58.1, U8.16
- new net N$113: C33.2, U8.19
- new net N$114: L6.2, L8.1, U8.12
- new net N$115: AE2.FEED, C38.2, C41.1
- new net N$116: C38.1, L7.2
- new net N$117: C39.1, C40.1, L8.2, U8.11
- new net N$118: C32.2, U7.VDD3P3/4, U7.VDD_RTC/5
- new net N$22: C29.2, L5.1, U7.LNA/2
- new net N$23: C27.1, U7.XTAL_OUT/27, Y3.1
- new net N$24: L3.1, U2.3
- new net N$25: C15.1, U2.1
- new net N$26: C13.2, R10.1, R13.2, U2.7
- new net N$27: R11.1, R14.2, U2.10
- new net N$28: LED3.A, R12.2
- new net N$30: R16.1, U3.23
- new net N$31: R17.1, U3.22
- new net N$32: R18.1, U4.24
- new net N$33: R19.1, U4.23
- new net N$34: R20.1, U4.22
- new net N$35: R15.1, U3.24
- new net N$36: DS9.R, R44.2
- new net N$37: DS7.R, R39.2
- new net N$38: DS7.B, R40.2
- new net N$39: DS7.G, R37.2
- new net N$40: DS9.B, R46.2
- new net N$41: DS9.G, R42.2
- new net N$42: DS2.G, R25.2
- new net N$43: DS2.B, R22.2
- new net N$44: DS11.B, R51.2
- new net N$45: DS11.G, R48.2
- new net N$46: R21.1, U3.1
- new net N$47: DS3.R, R28.2
- new net N$48: R23.1, U3.2
- new net N$49: R24.1, U3.3
- new net N$50: DS10.B, R43.2
- new net N$51: DS1.R, R23.2
- new net N$52: DS4.R, R29.2
- new net N$53: DS1.B, R24.2
- new net N$54: DS1.G, R21.2
- new net N$55: DS3.B, R30.2
- new net N$56: DS3.G, R26.2
- new net N$57: DS12.G, R52.2
- new net N$58: DS6.B, R33.2
- new net N$59: DS8.G, R41.2
- new net N$60: R26.1, U3.4
- new net N$61: DS4.G, R31.2
- new net N$62: DS10.G, R47.2
- new net N$63: DS4.B, R27.2
- new net N$64: DS6.G, R36.2
- new net N$65: DS5.B, R35.2
- new net N$66: DS5.G, R32.2
- new net N$67: DS10.R, R45.2
- new net N$68: DS8.B, R38.2
- new net N$69: R28.1, U3.5
- new net N$70: DS12.B, R49.2
- new net N$71: R30.1, U3.6
- new net N$72: R32.1, U3.7
- new net N$73: R35.1, U3.8
- new net N$74: R37.1, U3.10
- new net N$75: R39.1, U3.11
- new net N$76: R40.1, U3.12
- new net N$77: R42.1, U3.13
- new net N$78: R44.1, U3.14
- new net N$79: R46.1, U3.15
- new net N$80: R48.1, U3.16
- new net N$81: R51.1, U3.17
- new net N$82: DS6.R, R34.2
- new net N$83: DS12.R, R50.2
- new net N$84: R22.1, U4.17
- new net N$85: R25.1, U4.16
- new net N$86: R27.1, U4.15
- new net N$87: R29.1, U4.14
- new net N$88: R31.1, U4.13
- new net N$89: R33.1, U4.12
- new net N$90: R34.1, U4.11
- new net N$91: R36.1, U4.10
- new net N$92: R38.1, U4.8
- new net N$93: R41.1, U4.7
- new net N$94: R43.1, U4.6
- new net N$95: R45.1, U4.5
- new net N$96: R47.1, U4.4
- new net N$97: R49.1, U4.3
- new net N$98: R50.1, U4.2
- new net N$99: R52.1, U4.1
- new net SCL: R4.2, U1.37, U3.19, U4.19, U5.23
- new net WP#: U6.3, U7.SD_DATA_3/19
- net 3.3V: now also C1.1, C16.1, C17.1, C18.1, C19.1, C20.1, C21.2, C22.1, C24.1, C25.1, C28.2, C30.2, C31.2, C34.1, C35.1, C36.1, C37.1, DS1.V, DS10.V, DS11.V, DS12.V, DS2.V, DS3.V, DS4.V, DS5.V, DS6.V, DS7.V, DS8.V, DS9.V, R1.1, R11.2, R12.1, R20.2, R54.2, TP12.TP, TP15.TP, TP19.TP, TP25.TP, TP3.TP, TP31.TP, TP6.TP, TP9.TP, U2.2, U3.21, U4.21, U5.1, U5.13, U5.8, U6.8, U7.VDD3P3/3, U7.VDDA/1, U7.VDDA/30, U7.VDDD/29, U7.VDDPST/11, U7.VDDPST/17, U8.15, U8.18, U8.7; no longer C103.1, C222.2, C234.1, C235.1, C336.1, C337.2, C424.2, C425.1, C501.1, C502.1, C505.1, C507.1, C7.1, R107.2, R109.1, R215.2, R522.2, R9.1, TP17.TP, TP22.TP, TP23.TP, TP28.TP, TP29.TP, TP34.TP, TP35.TP, TP4.TP, U$203.8, U$206.VDDA/30, U$206.VDDD/29, U$206.VDDPST/11, U$206.VDDPST/17, U$304.15, U$304.18, U$304.7, U$508.V, U$511.V, U$513.V, U$514.V, U$515.V, U$516.V, U$517.V, U$518.V, U$520.21, U$521.21, U102.2, U403.1, U403.13, U403.8
- net CE: now also U8.1; no longer U$304.1
- net CHIP_EN: now also U7.CHIP_EN/7; no longer U$206.CHIP_EN/7
- net CSN: now also U8.2; no longer U$304.2
- net FSYNC: now also U5.11; no longer U403.11
- net GND: now also C1.2, C14.2, C15.2, C16.2, C17.2, C18.2, C19.2, C20.2, C21.1, C22.2, C23.1, C24.2, C25.2, C26.2, C27.2, C28.1, C30.1, C31.1, C32.1, C33.1, C34.2, C35.2, C36.2, C37.2, C39.2, C40.2, C41.2, C42.2, C43.2, L4.2, L5.2, LED3.C, R13.1, R14.1, R15.2, R16.2, R17.2, R18.2, R19.2, R53.2, R56.1, R57.1, R58.2, R9.1, TP11.TP, TP14.TP, TP17.TP, TP23.TP, TP29.TP, TP35.TP, TP5.TP, TP8.TP, U2.11, U2.12, U2.13, U2.14, U2.15, U2.4, U2.9, U3.9, U4.9, U5.18, U5.20, U5.9, U6.4, U7.GND, U8.14, U8.17, U8.20, U8.8; no longer C101.2, C103.2, C104.2, C207.2, C222.1, C223.2, C226.1, C228.1, C233.1, C234.2, C235.2, C308.1, C309.2, C310.2, C312.2, C314.2, C315.2, C336.2, C337.1, C424.1, C425.2, C427.1, C501.2, C502.2, C505.2, C507.2, C7.2, L207.2, L208.2, LED101.C, R104.1, R106.1, R201.2, R205.1, R251.1, R3.1, R312.2, R519.2, R520.2, R521.2, R523.2, R524.2, TP1.TP, TP19.TP, TP21.TP, TP25.TP, TP27.TP, TP3.TP, TP31.TP, TP33.TP, U$203.4, U$206.GND, U$304.14, U$304.17, U$304.20, U$304.8, U$520.9, U$521.9, U102.11, U102.12, U102.13, U102.14, U102.15, U102.4, U102.9, U403.18, U403.20, U403.9
- net GPIO0: now also U7.GPIO0/15; no longer U$206.GPIO0/15
- net GPIO2: now also U7.GPIO2/14; no longer U$206.GPIO2/14
- net INT: now also U5.12; no longer U403.12
- net IRQ: now also U8.6; no longer U$304.6
- net MISO: now also U8.5; no longer U$304.5
- net MOSI: now also U8.4; no longer U$304.4
- net N$11: now also TP33.TP; no longer TP9.TP
- net N$12: now also TP22.TP; no longer TP5.TP
- net N$14: now also TP28.TP; no longer TP6.TP
- net N$15: now also TP34.TP; no longer TP10.TP
- net N$16: now also TP16.TP; no longer TP11.TP
- net N$17: now also TP7.TP; no longer TP12.TP
- net N$18: now also TP10.TP; no longer TP13.TP
- net N$19: now also TP13.TP; no longer TP14.TP
- net N$20: now also TP4.TP; no longer TP15.TP
- net N$21: now also TP1.TP; no longer TP16.TP
- net N$29: now also R2.2; no longer R7.2
- net N$3: now also R55.2, U7.SD_CLK/21; no longer U1.45, U403.22
- net N$4: now also C23.2, U5.10; no longer R8.2, U$520.19, U$521.19, U1.37, U403.23
- net N$5: now also TP21.TP; no longer TP7.TP
- net N$6: now also TP27.TP; no longer TP8.TP
- net N$7: now also R1.2; no longer R6.2
- net PTA0: now also R9.2; no longer R3.2
- net PTA1: now also R7.2; no longer R4.2
- net PTA3: now also R6.2; no longer R2.2
- net RESET_B: now also R8.2; no longer R5.2
- net SCK: now also U8.3; no longer U$304.3
- net SDA: now also R5.2, U3.20, U4.20, U5.24; no longer R9.2, U$520.20, U$521.20, U403.24
- net U0RX: now also U7.U0RXD/25; no longer U$206.U0RXD/25
- net U0TX: now also U7.U0TXD/26; no longer U$206.U0TXD/26
- net VDDA: now also C6.1, R3.1; no longer C1.1, R1.1
- net VREFH: now also C7.1, R3.2; no longer C6.1, R1.2
- net VREFL: now also C7.2; no longer C1.2
- net V_IN: now also C13.1, C14.1, L3.2, R10.2, U2.5, U2.6, U2.8; no longer C101.1, C102.1, L101.2, R103.2, U102.5, U102.6, U102.8
- net WIFI_RESET: now also R54.1, U7.EXT_RSTB/32; no longer R215.1, U$206.EXT_RSTB/32
- net XPD_DCDC: now also U7.XPD_DCDC/8; no longer U$206.XPD_DCDC/8

Commit message: Matched all parts to bom-ex db.
Parts:
- removed LED1, LED2, LED3: (no value), appfruits:LED-0603
- added DS13, DS14, DS15: LTST-C19FD1WT, led:LTST-C19FD1WT
- added TP37, TP38, TP39, TP40, TP41, TP42, TP43, TP44, TP45, TP46, TP47, TP48, TP49, TP50, TP51, TP52, TP53, TP54, TP55, TP56, TP57, TP58: TPPAD1-20, testpad:P1-20
- AE1, AE2: value ANTENNA2SMD -> 2450AT18A100E
- C1, C15, C2, C3, C36, C4, C7, C8: device appfruits:0603-CAP -> SparkFun-Capacitors:0402-CAP
- C10: device appfruits:0603-CAP -> SparkFun-Capacitors:0603-CAP
- C11, C14, C9: value 10uF -> 0.1uF; device appfruits:0603-CAP -> SparkFun-Capacitors:0402-CAP
- C12: value 10uF -> 22uF; device appfruits:0603-CAP -> SparkFun-Capacitors:1210
- C13: value 0.1uF -> 22uF; device appfruits:0603-CAP -> SparkFun-Capacitors:1210
- C16: value 22uF -> 10uF; device appfruits:0603-CAP -> SparkFun-Capacitors:0603-CAP
- C17: value 0.1uF -> 10uF; device appfruits:0603-CAP -> SparkFun-Capacitors:0603-CAP
- C18, C20: value 2.2uF -> 0.1 uF; device appfruits:0603-CAP -> SparkFun-Capacitors:0402-CAP
- C19: value 0.1uF -> 0.1 uF; device appfruits:0603-CAP -> SparkFun-Capacitors:0402-CAP
- C21, C25, C32: value .1 uF -> 10uF
- C22, C23, C31, C34, C35: value .1 uF -> 0.1 uF; device SparkFun-Capacitors:0603-CAP -> SparkFun-Capacitors:0402-CAP
- C24: value .1 uF -> 15 pF; device SparkFun-Capacitors:0603-CAP -> SparkFun-Capacitors:0402-CAP
- C26, C38, C40, C41, C42, C43: device SparkFun-Capacitors:0603-CAP -> SparkFun-Capacitors:0402-CAP
- C27: value 15 pF -> 0.1 uF; device SparkFun-Capacitors:0603-CAP -> SparkFun-Capacitors:0402-CAP
- C28: value .1 uF -> 5.6 pF; device SparkFun-Capacitors:0603-CAP -> SparkFun-Capacitors:0402-CAP
- C29: value 5.6 pF -> 0.1 uF; device SparkFun-Capacitors:0603-CAP -> SparkFun-Capacitors:0402-CAP
- C30: value 1 uF -> 0.1 uF; device SparkFun-Capacitors:0603-CAP -> SparkFun-Capacitors:0402-CAP
- C33: value 33 nF -> .033 uF; device SparkFun-Capacitors:0603-CAP -> SparkFun-Capacitors:0402-CAP
- C37, C5, C6: value 2.2uF -> 10uF; device appfruits:0603-CAP -> SparkFun-Capacitors:0603-CAP
- C39: value 2.2 nF -> 2200 pF; device SparkFun-Capacitors:0603-CAP -> SparkFun-Capacitors:0402-CAP
- DS1, DS2, DS3: value LTST-C19FD1WT -> LTST-C191TBKT; device led:LTST-C19FD1WT -> appfruits:LED-0603
- JP1: value (none) -> M20PTH
- R1, R10, R11, R12, R13, R14, R2, R3: device appfruits:0603-RES -> appfruits:_0402
- R15, R16, R17, R18, R19, R20: device SparkFun:0603-RES -> appfruits:_0402
- R21, R22, R23, R24, R25, R26, R27, R28, R29, R30, R31, R32, R33, R34, R35, R36, R37, R38, R39, R40, R41, R42, R43, R44, R45, R46, R47, R48, R49, R50, R51, R52: value (none) -> 86.6; device SparkFun:0402-RES -> appfruits:_0402
- R4, R5, R53, R54, R55, R56, R57, R58, R59: device SparkFun-Resistors:0603-RES -> appfruits:_0402
- R6, R7, R8, R9: value (none) -> 10k; device SparkFun:0402-RES -> appfruits:_0402
- S1: value (none) -> CUS-12TB
- Y1: value 16Mhz/8pF -> 8MHz; device appfruits:CRYSTAL-SMD-5X3 -> CrystalOscillators:ASCO
- Y2: value 32.768KHz -> 34.728kHz; device appfruits:CRYSTAL-TXC-7A -> CrystalOscillators:ABS06
- moved U7 425.1 mm to (40.6, 41.9)
- moved U8 409.0 mm to (11.4, 11.4), turned to 90 degrees
- moved U5 404.2 mm to (41.9, 26.7)
- moved DS3 390.6 mm to (-49.5, 34.3)
- moved U4 384.7 mm to (24.1, 41.9)
- moved DS5 367.2 mm to (-30.5, 8.89)
- moved DS1 367.1 mm to (43.2, -6.35)
- moved C24 366.2 mm to (-40.6, -12.7)
- moved C28 366.2 mm to (-48.3, -12.7)
- moved DS10 365.5 mm to (-33.0, 8.89)
- moved DS12 365.1 mm to (-35.6, 8.89)
- moved C31 363.0 mm to (-45.7, -16.5)
- moved C34 362.8 mm to (-45.7, -41.9)
- moved C35 362.8 mm to (-49.5, -41.9)
- moved L6 362.8 mm to (-45.7, -45.7)
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Connections:
- net !CS: now also TP44.TP
- net !RESET0: now also TP39.TP
- net !RESET1: now also TP40.TP
- net 3.3V: now also C12.1, C13.1, C14.1, C15.1, C18.2, C21.1, C23.1, C27.2, C29.2, C32.1, DS13.V, DS14.V, DS15.V, Y1.VCC; no longer C18.1, C20.1, C21.2, C24.1, C28.2, C31.2, DS1.V, DS2.V, DS3.V
- net CE: now also TP58.TP
- net CHIP_EN: now also TP50.TP
- net CSN: now also TP57.TP
- net FSYNC: now also TP41.TP
- net GND: now also C10.2, C11.2, C12.2, C13.2, C18.1, C20.1, C21.2, C23.2, C27.1, C29.1, C32.2, DS3.C, Y1.GND; no longer C10.1, C11.1, C12.1, C18.2, C20.2, C21.1, C23.1, C27.2, C28.1, C32.1, C9.1, LED3.C
- net GPIO0: now also TP52.TP
- net GPIO2: now also TP51.TP
- net INT: now also TP45.TP
- net IRQ: now also TP53.TP
- net MISO: now also TP54.TP
- net MOSI: now also TP55.TP
- net N$1: now also U1.32, Y1.OUT; no longer C11.2, U1.19, Y2.P$2
- net N$10: now also DS1.C; no longer LED1.C
- net N$100: now also C24.1; no longer C26.1
- net N$101: now also C28.1; no longer C29.1
- net N$118: now also C31.2; no longer C32.2
- net N$13: now also DS2.C; no longer LED2.C
- net N$2: now also U1.33, Y1.ENABLE; no longer C12.2, U1.20, Y2.P$1
- net N$22: now also C28.2; no longer C29.2
- net N$23: now also C26.1; no longer C27.1
- net N$25: now also C11.1; no longer C15.1
- net N$26: now also C9.2; no longer C13.2
- net N$28: now also DS3.A; no longer LED3.A
- net N$29: now also DS2.A; no longer LED2.A
- net N$36: now also DS12.R; no longer DS9.R
- net N$37: now also DS10.R; no longer DS7.R
- net N$38: now also DS10.B; no longer DS7.B
- net N$39: now also DS10.G; no longer DS7.G
- net N$4: now also C20.2; no longer C23.2
- net N$40: now also DS12.B; no longer DS9.B
- net N$41: now also DS12.G; no longer DS9.G
- net N$42: now also DS5.G; no longer DS2.G
- net N$43: now also DS5.B; no longer DS2.B
- net N$44: now also DS14.B; no longer DS11.B
- net N$45: now also DS14.G; no longer DS11.G
- net N$47: now also DS6.R; no longer DS3.R
- net N$50: now also DS13.B; no longer DS10.B
- net N$51: now also DS4.R; no longer DS1.R
- net N$52: now also DS7.R; no longer DS4.R
- net N$53: now also DS4.B; no longer DS1.B
- net N$54: now also DS4.G; no longer DS1.G
- net N$55: now also DS6.B; no longer DS3.B
- net N$56: now also DS6.G; no longer DS3.G
- net N$57: now also DS15.G; no longer DS12.G
- net N$58: now also DS9.B; no longer DS6.B
- net N$59: now also DS11.G; no longer DS8.G
- net N$61: now also DS7.G; no longer DS4.G
- net N$62: now also DS13.G; no longer DS10.G
- net N$63: now also DS7.B; no longer DS4.B
- net N$64: now also DS9.G; no longer DS6.G
- net N$65: now also DS8.B; no longer DS5.B
- net N$66: now also DS8.G; no longer DS5.G
- net N$67: now also DS13.R; no longer DS10.R
- net N$68: now also DS11.B; no longer DS8.B
- net N$7: now also DS1.A; no longer LED1.A
- net N$70: now also DS15.B; no longer DS12.B
- net N$8: now also U1.19, Y2.P$2; no longer C9.2, U1.32, Y1.3
- net N$82: now also DS9.R; no longer DS6.R
- net N$83: now also DS15.R; no longer DS12.R
- net N$9: now also U1.20, Y2.P$1; no longer C10.2, U1.33, Y1.1
- net SCK: now also TP56.TP
- net SCL: now also R5.2, TP42.TP; no longer R4.2
- net SDA: now also R4.2, TP37.TP, TP38.TP, TP43.TP; no longer R5.2
- net U0RX: now also TP47.TP
- net U0TX: now also TP46.TP
- net V_IN: now also C10.1, C9.1; no longer C13.1, C14.1
- net WIFI_RESET: now also TP48.TP
- net XPD_DCDC: now also TP49.TP
Other:
- board size 160 x 100 mm -> 50.8 x 50.8 mm

Commit message: Began laying out PCB
Parts:
- removed C42, C43: 22 pF, SparkFun-Capacitors:0402-CAP
- C10: value 10uF -> 22uF; device SparkFun-Capacitors:0603-CAP -> SparkFun-Capacitors:1210
- C11: value 0.1uF -> 22uF; device SparkFun-Capacitors:0402-CAP -> SparkFun-Capacitors:1210
- C12, C13: value 22uF -> 0.1uF; device SparkFun-Capacitors:1210 -> SparkFun-Capacitors:0402-CAP
- C14, C15, C4, C8: value 0.1uF -> 10uF; device SparkFun-Capacitors:0402-CAP -> SparkFun-Capacitors:0603-CAP
- C16, C17, C21, C25, C32: value 10uF -> 0.1 uF; device SparkFun-Capacitors:0603-CAP -> SparkFun-Capacitors:0402-CAP
- C19, C23, C30, C35: value 0.1 uF -> 10uF; device SparkFun-Capacitors:0402-CAP -> SparkFun-Capacitors:0603-CAP
- C22: value 0.1 uF -> 15 pF
- C26: value 15 pF -> 5.6 pF
- C28: value 5.6 pF -> 0.1 uF
- C31: value 0.1 uF -> .033 uF
- C33: value .033 uF -> 0.1 uF
- C34: value 0.1 uF -> 0.1uF
- C36: value 0.1uF -> 1.5 pF
- C37: value 10uF -> 2200 pF; device SparkFun-Capacitors:0603-CAP -> SparkFun-Capacitors:0402-CAP
- C38: value 1.5 pF -> 4.7 pF
- C39: value 2200 pF -> 1.0 pF
- C40: value 4.7 pF -> 22 pF
- C41: value 1.0 pF -> 22 pF
- C6: value 10uF -> 0.1uF; device SparkFun-Capacitors:0603-CAP -> SparkFun-Capacitors:0402-CAP
- JP1: device SparkFun-Connectors:1X02 -> SparkFun-Connectors:JST_2PIN
- R1, R12, R2: value 470 -> 25
- R11: value 1.2M -> 220K
- R13: value 220K -> 1.2M
- moved U7 93.1 mm to (-52.2, 34.5)
- moved U5 88.0 mm to (-40.1, 58.5)
- moved C25 80.4 mm to (-38.1, 37.3)
- moved C21 75.6 mm to (-34.3, 37.3)
- moved C29 71.4 mm to (-41.9, 37.3)
- moved C19 71.1 mm to (15.2, -31.8)
- moved C34 69.0 mm to (-33.0, 25.9)
- moved C9 67.2 mm to (17.5, 45.6), turned to 270 degrees
- moved C30 65.8 mm to (15.2, -27.9)
- moved C11 65.3 mm to (19.4, 45.6), turned to 270 degrees
- moved R13 64.5 mm to (18.7, 42.4)
- moved C10 64.2 mm to (22.2, 45.6), turned to 270 degrees
- moved L3 62.9 mm to (13.3, 48.6), turned to 180 degrees
- moved R10 62.3 mm to (12.7, 41.4), turned to 180 degrees
- moved C35 61.6 mm to (-45.7, 19.6)
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Connections:
- removed net N$110: JP1.1, S1.3
- new net N$104: JP1.1, S1.2
- net 3.3V: now also C10.1, C11.1, C16.2, C20.1, C25.2, C28.2, C30.1, C33.1, R13.2; no longer C16.1, C18.2, C22.1, C25.1, C29.2, C30.2, C36.1, C37.1, C5.1, R11.2
- net GND: now also C16.1, C20.2, C25.1, C28.1, C30.2, C33.2, C38.2, C8.2, C9.2, R11.1; no longer C16.2, C20.1, C25.2, C26.2, C30.1, C33.1, C36.2, C42.2, C43.2, C5.2, R13.1
- net N$100: now also C22.1; no longer C24.1
- net N$101: now also C26.1; no longer C28.1
- net N$108: now also C40.1; no longer C42.1
- net N$109: now also C41.1; no longer C43.1
- net N$113: now also C31.2; no longer C33.2
- net N$115: now also C36.2, C39.1; no longer C38.2, C41.1
- net N$116: now also C36.1; no longer C38.1
- net N$117: now also C37.1, C38.1; no longer C39.1, C40.1
- net N$118: now also C29.2; no longer C31.2
- net N$22: now also C26.2; no longer C28.2
- net N$23: now also C24.1; no longer C26.1
- net N$25: now also C9.1; no longer C11.1
- net N$26: now also R11.2; no longer C9.2, R13.2
- net N$27: now also R13.1; no longer R11.1
- net N$4: now also C18.2; no longer C20.2
- net VDDA: now also C5.1; no longer C6.1
- net VREFH: now also C6.1; no longer C7.1
- net VREFL: now also C5.2; no longer C8.2
- net VREF_OUT: now also C7.1; no longer C8.1
- net V_IN: now also C8.1, S1.3; no longer C10.1, C9.1, S1.2
Routing:
- added copper zone on layer 15, net 3.3V
- added copper zone on layer 1, net GND
- added copper zone on layer 16, net GND
- added copper zone on layer 2, net GND
